File: hardware/kicad/tinyscope/tinyscope.kicad_sch (KiCad schematic)
At the start: 0 parts

Commit message: feat: hardware: Add tinyscope kicad project. Create flow diagram on Power Input & Charging schemat
Other:
- added sheet Front End (front_end.kicad_sch)
- added sheet HMI (hmi.kicad_sch)
- note added: "---------------------------->"
- note added: "----->"
- note added: "-->"
- note added: "<-"
Changed lines of the file:
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@@
 (kicad_sch (version 20230121) (generator eeschema)
-  (paper "A3")
+  (paper "A4")
   (title_block
     (title "tinyscope")
@@
     (rev "0.1")
   )
-  (sheet (at 355.6 147.32) (size 17.78 7.62) (fields_autoplaced)
+  (text "<-" (at 246.38 35.56 90)
+    (effects (font (size 2.5 2.5) (thickness 0.7) bold (color 0 0 0 1)) (justify left bottom))
+  )
+  (text "---------------------------->" (at 64.262 26.924 0)
+    (effects (font (size 2.5 2.5) (thickness 0.7) bold (color 0 0 0 1)) (justify left bottom))
+  )
+  (text "-->" (at 61.976 52.324 0)
+    (effects (font (size 2.5 2.5) (thickness 0.7) bold (color 0 0 0 1)) (justify left bottom))
+  )
+  (text "-->" (at 225.552 27.178 0)
+    (effects (font (size 2.5 2.5) (thickness 0.7) bold (color 0 0 0 1)) (justify right bottom))
+  )
+  (text "<-" (at 246.38 48.26 90)
+    (effects (font (size 2.5 2.5) (thickness 0.7) bold (color 0 0 0 1)) (justify left bottom))
+  )
+  (text "----->" (at 182.88 48.26 90)
+    (effects (font (size 2.5 2.5) (thickness 0.7) bold (color 0 0 0 1)) (justify left bottom))
+  )
+  (text "-->" (at 147.066 52.324 0)
+    (effects (font (size 2.5 2.5) (thickness 0.7) bold (color 0 0 0 1)) (justify left bottom))
+  )
+  (sheet (at 66.04 149.86) (size 17.78 7.62) (fields_autoplaced)
     (stroke (width 0.1524) (type solid))
     (fill (color 0 0 0 0.0000))
-    (property "Sheetname" "Regulation & Rails" (at 355.6 146.6084 0)
-      (effects (font (size 1.27 1.27)) (justify left bottom))
+    (property "Sheetname" "Regulation & Rails" (at 66.04 148.5334 0)
+      (effects (font (size 2.5 2.5) bold) (justify left bottom))
     )
-    (property "Sheetfile" "regulation_and_rails.kicad_sch" (at 355.6 155.5246 0)
-      (effects (font (size 1.27 1.27)) (justify left top))
+    (property "Sheetfile" "regulation_and_rails.kicad_sch" (at 66.04 158.0646 0)
+      (effects (font (size 1.27 1.27)) (justify left top) hide)
     )
     (instances
@@
     )
   )
-  (sheet (at 317.5 144.78) (size 22.86 10.16)
+  (sheet (at 119.38 137.16) (size 12.7 5.08) (fields_autoplaced)
     (stroke (width 0.1524) (type solid))
     (fill (color 255 255 194 1.0000))
-    (property "Sheetname" "Power Input & Charging" (at 317.5 144.0684 0)
+    (property "Sheetname" "Front End" (at 119.38 136.4484 0)
       (effects (font (size 1.27 1.27)) (justify left bottom))
     )
-    (property "Sheetfile" "power_and_charging.kicad_sch" (at 317.5 155.5246 0)
+    (property "Sheetfile" "front_end.kicad_sch" (at 119.38 142.8246 0)
       (effects (font (size 1.27 1.27)) (justify left top))
     )
-    (property "USBC" "USBC" (at 322.58 147.32 0)
-      (effects (font (size 1.27 1.27)))
+    (instances
+      (project "tinyscope"
+        (path "/bb072e32-cc57-415a-8554-0e84d374f333" (page "5"))
+      )
+    )
+  )
+  (sheet (at 17.78 20.32) (size 261.62 35.56)
+    (stroke (width 0.1524) (type solid))
+    (fill (color 255 255 194 1.0000))
+    (property "Sheetname" "Power Input & Charging" (at 17.78 19.6084 0)
+      (effects (font (size 2.5 2.5) bold) (justify left bottom))
+    )
+    (property "Sheetfile" "power_and_charging.kicad_sch" (at 17.78 31.0646 0)
+      (effects (font (size 1.27 1.27)) (justify left top) hide)
+    )
+    (property "USBC" "Power Input 5V" (at 40.64 25.4 0) (show_name)
+      (effects (font (size 2.5 2.5) bold))
+    )
+    (property "Schottkey OR" "Source OR-ing" (at 185.42 25.4 0) (show_name)
+      (effects (font (size 2.5 2.5) bold))
+    )
+    (property "BQ24075" "Charger" (at 243.84 25.4 0) (show_name)
+      (effects (font (size 2.5 2.5) bold))
+    )
+    (property "External Battery" "12V" (at 40.64 50.8 0) (show_name)
+      (effects (font (size 2.5 2.5) bold))
+    )
+    (property "Input Protection" "Fuse->P-FET->TVS" (at 109.22 50.8 0) (show_name)
+      (effects (font (size 2.5 2.5) bold))
+    )
+    (property "TPS54360" "Buck Converter" (at 182.88 50.8 0) (show_name)
+      (effects (font (size 2.5 2.5) bold))
+    )
+    (property "Device Battery" "1S LiPo" (at 248.92 38.1 0) (show_name)
+      (effects (font (size 2.5 2.5) bold))
+    )
+    (property "MAX17048" "Fuel Gauge" (at 248.92 50.8 0) (show_name)
+      (effects (font (size 2.5 2.5) bold))
     )
     (instances
@@
     )
   )
-  (sheet (at 317.5 177.8) (size 12.7 5.08) (fields_autoplaced)
+  (sheet (at 152.4 121.92) (size 12.7 5.08) (fields_autoplaced)
+    (stroke (width 0.1524) (type solid))
+    (fill (color 255 255 194 1.0000))
+    (property "Sheetname" "HMI" (at 152.4 121.2084 0)
+      (effects (font (size 1.27 1.27)) (justify left bottom))
+    )
+    (property "Sheetfile" "hmi.kicad_sch" (at 152.4 127.5846 0)
+      (effects (font (size 1.27 1.27)) (justify left top))
+    )
+    (instances
+      (project "tinyscope"
+        (path "/bb072e32-cc57-415a-8554-0e84d374f333" (page "6"))
+      )
+    )
+  )
+  (sheet (at 109.22 106.68) (size 12.7 5.08) (fields_autoplaced)
     (stroke (width 0.1524) (type solid))
     (fill (color 0 0 0 0.0000))
-    (property "Sheetname" "MCUS" (at 317.5 177.0884 0)
+    (property "Sheetname" "MCUS" (at 109.22 105.9684 0)
       (effects (font (size 1.27 1.27)) (justify left bottom))
     )
-    (property "Sheetfile" "mcus.kicad_sch" (at 317.5 183.4646 0)
+    (property "Sheetfile" "mcus.kicad_sch" (at 109.22 112.3446 0)
       (effects (font (size 1.27 1.27)) (justify left top))
     )
