File: hardware/kicad/tinyscope/mcu_wireless.kicad_sch (KiCad schematic)
At the start: 13 parts, among them J4 MDBT50Q_TAG_CONNECT, Q2 NMOS, U11 MDBT50Q-1MV2, X1 32k768

Commit message: feat: hardware: Adds SPI4 connection on wireless mcu schematic
Connections:
- net STM32H743_SPI1_IRQ renamed STM32H743_SPI4_IRQ
- net STM32H743_SPI1_MISO renamed STM32H743_SPI4_MISO
- net STM32H743_SPI1_MOSI renamed STM32H743_SPI4_MOSI
- net STM32H743_SPI1_NSS renamed STM32H743_SPI4_NSS
- net STM32H743_SPI1_SCK renamed STM32H743_SPI4_SCK
Changed lines of the file:
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@@
     (effects (font (size 1.27 1.27)) (justify left top))
   )
-  (label "STM32H743_SPI1_MISO" (at 203.2 109.22 180) (fields_autoplaced)
+  (label "STM32H743_SPI4_MISO" (at 203.2 109.22 180) (fields_autoplaced)
     (effects (font (size 1.27 1.27) bold) (justify right bottom))
   )
-  (label "STM32H743_SPI1_SCK" (at 203.2 101.6 180) (fields_autoplaced)
+  (label "STM32H743_SPI4_SCK" (at 203.2 101.6 180) (fields_autoplaced)
     (effects (font (size 1.27 1.27) bold) (justify right bottom))
   )
-  (label "STM32H743_SPI1_IRQ" (at 203.2 104.14 180) (fields_autoplaced)
+  (label "STM32H743_SPI4_IRQ" (at 203.2 104.14 180) (fields_autoplaced)
     (effects (font (size 1.27 1.27) bold) (justify right bottom))
   )
@@
     (effects (font (size 1.27 1.27) bold) (justify left bottom))
   )
-  (label "STM32H743_SPI1_NSS" (at 203.2 106.68 180) (fields_autoplaced)
+  (label "STM32H743_SPI4_NSS" (at 203.2 106.68 180) (fields_autoplaced)
     (effects (font (size 1.27 1.27) bold) (justify right bottom))
   )
@@
     (effects (font (size 1.27 1.27) bold) (justify left bottom))
   )
-  (label "STM32H743_SPI1_MOSI" (at 203.2 111.76 180) (fields_autoplaced)
+  (label "STM32H743_SPI4_MOSI" (at 203.2 111.76 180) (fields_autoplaced)
     (effects (font (size 1.27 1.27) bold) (justify right bottom))
   )
