File: hardware/kicad/tinyscope/mcus_acquisition.kicad_sch (KiCad schematic)
At the start: 30 parts, among them J5 STM32H743, Q2 NMOS, SW1 SW_SPST, U12 STM32H743VITx, X1 25MHz, X2 32k768

Commit message: fix: hardware: Solves electrical rules warnings and errors #2
Connections:
- net ENC6_A: now also U12.82 (PD1)
- net ENC6_B: now also U12.83 (PD2)
- net ENC6_SW: now also U12.81 (PD0)
- net STM32H743_USB_DM: now reaches U12.70 (PA11)
- net STM32H743_USB_DP: now reaches U12.71 (PA12)
- net MAX17048_ALRTB: now reaches U12.86 (PD5)
- net STM32H743_I2C1_SCL: now reaches U12.92 (PB6)
- net STM32H743_I2C1_SDA: now reaches U12.93 (PB7)
Other:
- note removed: "Find the place for the encoder 6th"
- moved on the sheet: J5
Changed lines of the file:
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@@
     (stroke (width 0) (type default))
   )
-  (wire (pts (xy 223.52 71.12) (xy 203.2 71.12))
+  (wire (pts (xy 231.14 71.12) (xy 210.82 71.12))
     (stroke (width 0) (type default))
   )
@@
     (stroke (width 0) (type default))
   )
-  (wire (pts (xy 200.66 60.96) (xy 223.52 60.96))
+  (wire (pts (xy 208.28 60.96) (xy 231.14 60.96))
     (stroke (width 0) (type default))
   )
@@
     (stroke (width 0) (type default))
   )
+  (wire (pts (xy 177.8 66.04) (xy 203.2 66.04))
+    (stroke (width 0) (type default))
+  )
   (wire (pts (xy 43.18 43.18) (xy 43.18 45.72))
     (stroke (width 0) (type default))
@@
     (stroke (width 0) (type default))
   )
-  (wire (pts (xy 233.68 53.34) (xy 233.68 55.88))
+  (wire (pts (xy 241.3 53.34) (xy 241.3 55.88))
     (stroke (width 0) (type default))
   )
@@
     (stroke (width 0) (type default))
   )
-  (wire (pts (xy 259.08 99.06) (xy 236.22 99.06))
+  (wire (pts (xy 134.62 101.6) (xy 111.76 101.6))
     (stroke (width 0) (type default))
   )
@@
     (stroke (width 0) (type default))
   )
-  (wire (pts (xy 177.8 68.58) (xy 223.52 68.58))
-    (stroke (width 0) (type default))
-  )
   (wire (pts (xy 43.18 20.32) (xy 43.18 22.86))
     (stroke (width 0) (type default))
@@
     (stroke (width 0) (type default))
   )
-  (wire (pts (xy 203.2 71.12) (xy 203.2 86.36))
+  (wire (pts (xy 210.82 71.12) (xy 210.82 86.36))
+    (stroke (width 0) (type default))
+  )
+  (wire (pts (xy 177.8 68.58) (xy 231.14 68.58))
     (stroke (width 0) (type default))
   )
@@
     (stroke (width 0) (type default))
   )
-  (wire (pts (xy 223.52 66.04) (xy 200.66 66.04))
+  (wire (pts (xy 231.14 66.04) (xy 208.28 66.04))
     (stroke (width 0) (type default))
   )
@@
     (stroke (width 0) (type default))
   )
+  (wire (pts (xy 177.8 63.5) (xy 203.2 63.5))
+    (stroke (width 0) (type default))
+  )
   (wire (pts (xy 160.02 25.4) (xy 162.56 25.4))
     (stroke (width 0) (type default))
@@
     (stroke (width 0) (type default))
   )
+  (wire (pts (xy 111.76 114.3) (xy 134.62 114.3))
+    (stroke (width 0) (type default))
+  )
   (wire (pts (xy 109.22 48.26) (xy 104.14 48.26))
     (stroke (width 0) (type default))
@@
     (stroke (width 0) (type default))
   )
-  (wire (pts (xy 233.68 76.2) (xy 233.68 78.74))
+  (wire (pts (xy 241.3 76.2) (xy 241.3 78.74))
     (stroke (width 0) (type default))
   )
@@
     (stroke (width 0) (type default))
   )
-  (wire (pts (xy 200.66 66.04) (xy 200.66 71.12))
+  (wire (pts (xy 208.28 66.04) (xy 208.28 71.12))
     (stroke (width 0) (type default))
   )
@@
     (stroke (width 0) (type default))
   )
-  (wire (pts (xy 259.08 101.6) (xy 236.22 101.6))
-    (stroke (width 0) (type default))
-  )
-  (wire (pts (xy 259.08 104.14) (xy 236.22 104.14))
+  (wire (pts (xy 134.62 104.14) (xy 111.76 104.14))
+    (stroke (width 0) (type default))
+  )
+  (wire (pts (xy 177.8 96.52) (xy 203.2 96.52))
+    (stroke (width 0) (type default))
+  )
+  (wire (pts (xy 134.62 106.68) (xy 111.76 106.68))
     (stroke (width 0) (type default))
   )
@@
     (stroke (width 0) (type default))
   )
-  (wire (pts (xy 200.66 71.12) (xy 177.8 71.12))
+  (wire (pts (xy 208.28 71.12) (xy 177.8 71.12))
     (stroke (width 0) (type default))
   )
@@
     (stroke (width 0) (type default))
   )
+  (wire (pts (xy 177.8 93.98) (xy 203.2 93.98))
+    (stroke (width 0) (type default))
+  )
   (wire (pts (xy 53.34 48.26) (xy 53.34 45.72))
     (stroke (width 0) (type default))
@@
     (stroke (width 0) (type default))
   )
-  (wire (pts (xy 203.2 86.36) (xy 177.8 86.36))
+  (wire (pts (xy 210.82 86.36) (xy 177.8 86.36))
     (stroke (width 0) (type default))
   )
@@
     (effects (font (size 1.27 1.27) (thickness 0.254) bold) (justify left top))
   )
-  (text "Find the place for the encoder 6th" (at 236.22 91.44 0)
-    (effects (font (size 1.27 1.27)) (justify left bottom))
-  )
   (label "STM32H743_SWD_NRST" (at 113.03 25.4 0) (fields_autoplaced)
     (effects (font (size 1.27 1.27) bold) (justify left bottom))
@@
     (effects (font (size 1.27 1.27) bold) (justify right bottom))
   )
+  (label "MAX17048_ALRTB" (at 111.76 114.3 0) (fields_autoplaced)
+    (effects (font (size 1.27 1.27) bold) (justify left bottom))
+  )
   (label "STM32H743_SPI2_NSS" (at 203.2 109.22 180) (fields_autoplaced)
     (effects (font (size 1.27 1.27) bold) (justify right bottom))
@@
     (effects (font (size 1.27 1.27) bold) (justify right bottom))
   )
+  (label "STM32H743_USB_DP" (at 203.2 66.04 180) (fields_autoplaced)
+    (effects (font (size 1.27 1.27) bold) (justify right bottom))
+  )
   (label "ENC1_SW" (at 203.2 40.64 180) (fields_autoplaced)
     (effects (font (size 1.27 1.27) bold) (justify right bottom))
@@
     (effects (font (size 1.27 1.27) bold) (justify left bottom))
   )
-  (label "STM32H743_SWD_NRST" (at 200.66 60.96 0) (fields_autoplaced)
+  (label "STM32H743_SWD_NRST" (at 208.28 60.96 0) (fields_autoplaced)
     (effects (font (size 1.27 1.27) bold) (justify left bottom))
   )
@@
     (effects (font (size 1.27 1.27) bold) (justify right bottom))
   )
-  (label "ENC6_SW" (at 236.22 99.06 0) (fields_autoplaced)
+  (label "STM32H743_I2C1_SDA" (at 203.2 96.52 180) (fields_autoplaced)
+    (effects (font (size 1.27 1.27) bold) (justify right bottom))
+  )
+  (label "ENC6_SW" (at 111.76 101.6 0) (fields_autoplaced)
     (effects (font (size 1.27 1.27) bold) (justify left bottom))
   )
@@
     (effects (font (size 1.27 1.27) bold) (justify left bottom))
   )
-  (label "ENC6_A" (at 236.22 101.6 0) (fields_autoplaced)
+  (label "ENC6_A" (at 111.76 104.14 0) (fields_autoplaced)
     (effects (font (size 1.27 1.27) bold) (justify left bottom))
   )
@@
     (effects (font (size 1.27 1.27) bold) (justify right bottom))
   )
+  (label "STM32H743_USB_DM" (at 203.2 63.5 180) (fields_autoplaced)
+    (effects (font (size 1.27 1.27) bold) (justify right bottom))
+  )
   (label "ENC2_B" (at 111.76 86.36 0) (fields_autoplaced)
     (effects (font (size 1.27 1.27) bold) (justify left bottom))
@@
     (effects (font (size 1.27 1.27) bold) (justify right bottom))
   )
-  (label "ENC6_B" (at 236.22 104.14 0) (fields_autoplaced)
-    (effects (font (size 1.27 1.27) bold) (justify left bottom))
+  (label "ENC6_B" (at 111.76 106.68 0) (fields_autoplaced)
+    (effects (font (size 1.27 1.27) bold) (justify left bottom))
+  )
+  (label "STM32H743_I2C1_SCL" (at 203.2 93.98 180) (fields_autoplaced)
+    (effects (font (size 1.27 1.27) bold) (justify right bottom))
   )
   (label "ENC2_A" (at 111.76 81.28 0) (fields_autoplaced)
@@
     )
   )
-  (symbol (lib_id "power:GND") (at 233.68 78.74 0) (mirror y) (unit 1)
+  (symbol (lib_id "power:GND") (at 241.3 78.74 0) (mirror y) (unit 1)
     (in_bom yes) (on_board yes) (dnp no) (fields_autoplaced)
-    (property "Reference" "#PWR?" (at 233.68 85.09 0)
-      (effects (font (size 1.27 1.27)) hide)
-    )
-    (property "Value" "GND" (at 233.68 83.82 0)
-      (effects (font (size 1.27 1.27)) hide)
-    )
-    (property "Footprint" "" (at 233.68 78.74 0)
-      (effects (font (size 1.27 1.27)) hide)
-    )
-    (property "Datasheet" "" (at 233.68 78.74 0)
+    (property "Reference" "#PWR?" (at 241.3 85.09 0)
+      (effects (font (size 1.27 1.27)) hide)
+    )
+    (property "Value" "GND" (at 241.3 83.82 0)
+      (effects (font (size 1.27 1.27)) hide)
+    )
+    (property "Footprint" "" (at 241.3 78.74 0)
+      (effects (font (size 1.27 1.27)) hide)
+    )
+    (property "Datasheet" "" (at 241.3 78.74 0)
       (effects (font (size 1.27 1.27)) hide)
     )
@@
     )
   )
-  (symbol (lib_id "Connector:Conn_ARM_SWD_TagConnect_TC2030-NL") (at 231.14 66.04 0) (mirror y) (unit 1)
+  (symbol (lib_id "Connector:Conn_ARM_SWD_TagConnect_TC2030-NL") (at 238.76 66.04 0) (mirror y) (unit 1)
     (in_bom no) (on_board yes) (dnp no)
-    (property "Reference" "J5" (at 226.06 57.15 0)
-      (effects (font (size 1.27 1.27)) (justify right))
-    )
-    (property "Value" "STM32H743" (at 220.345 74.93 0)
-      (effects (font (size 1.27 1.27)) (justify right))
-    )
-    (property "Footprint" "Connector:Tag-Connect_TC2030-IDC-NL_2x03_P1.27mm_Vertical" (at 231.14 83.82 0)
-      (effects (font (size 1.27 1.27)) hide)
-    )
-    (property "Datasheet" "https://www.tag-connect.com/wp-content/uploads/bsk-pdf-manager/TC2030-CTX_1.pdf" (at 231.14 81.28 0)
+    (property "Reference" "J5" (at 233.68 57.15 0)
+      (effects (font (size 1.27 1.27)) (justify right))
+    )
+    (property "Value" "STM32H743" (at 227.965 74.93 0)
+      (effects (font (size 1.27 1.27)) (justify right))
+    )
+    (property "Footprint" "Connector:Tag-Connect_TC2030-IDC-NL_2x03_P1.27mm_Vertical" (at 238.76 83.82 0)
+      (effects (font (size 1.27 1.27)) hide)
+    )
+    (property "Datasheet" "https://www.tag-connect.com/wp-content/uploads/bsk-pdf-manager/TC2030-CTX_1.pdf" (at 238.76 81.28 0)
       (effects (font (size 1.27 1.27)) hide)
     )
@@
     )
   )
-  (symbol (lib_id "power:+3V3") (at 233.68 53.34 0) (mirror y) (unit 1)
-    (in_bom yes) (on_board yes) (dnp no)
-    (property "Reference" "#PWR063" (at 233.68 57.15 0)
-      (effects (font (size 1.27 1.27)) hide)
-    )
-    (property "Value" "+3V3" (at 233.045 49.53 0)
+  (symbol (lib_id "power:+3V3") (at 241.3 53.34 0) (mirror y) (unit 1)
+    (in_bom yes) (on_board yes) (dnp no)
+    (property "Reference" "#PWR063" (at 241.3 57.15 0)
+      (effects (font (size 1.27 1.27)) hide)
+    )
+    (property "Value" "+3V3" (at 240.665 49.53 0)
       (effects (font (size 1.27 1.27)))
     )
-    (property "Footprint" "" (at 233.68 53.34 0)
-      (effects (font (size 1.27 1.27)) hide)
-    )
-    (property "Datasheet" "" (at 233.68 53.34 0)
-      (effects (font (size 1.27 1.27)) hide)
-    )
+    (property "Footprint" "" (at 241.3 53.34 0)
+      (effects (font (size 1.27 1.27)) hide)
+    )
+    (property "Datasheet" "" (at 241.3 53.34 0)
+      (effects (font (size 1.27 1.27)) hide)
+    )
