File: hardware/kicad/tinyscope/mcus_acquisition.kicad_sch (KiCad schematic)
At the start: 30 parts, among them J5 STM32H743, Q2 NMOS, SW1 SW_SPST, U12 STM32H743VITx, X1 25MHz, X2 32k768

Commit message: feat: hardware: Maps waveshare display connections
Connections:
- net STM32H743_GPIO_EXTI1: now also U12.16 (PC1)
- net STM32H743_I2C1_SCL: now also U12.95 (PB8); no longer U12.92 (PB6)
- net STM32H743_GPIO_OUT_PC0: now reaches U12.15 (PC0)
- new net STM32H743_TIM4_CH1: U12.92 (PB6)
- no-connect marks 38 -> 35
Changed lines of the file:
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@@
   (junction (at 104.14 20.32) (diameter 0) (color 0 0 0 0)
   )
-  (no_connect (at 177.8 124.46))
   (no_connect (at 134.62 66.04))
   (no_connect (at 177.8 129.54))
@@
   (no_connect (at 177.8 154.94))
   (no_connect (at 177.8 83.82))
-  (no_connect (at 177.8 99.06))
   (no_connect (at 134.62 78.74))
   (no_connect (at 177.8 60.96))
@@
   (no_connect (at 134.62 127))
   (no_connect (at 177.8 101.6))
-  (no_connect (at 177.8 121.92))
   (no_connect (at 177.8 73.66))
   (no_connect (at 134.62 119.38))
@@
     )
   )
-  (global_label "STM32H743_I2C1_SCL" (shape bidirectional) (at 177.8 93.98 0) (fields_autoplaced)
-    (effects (font (size 1.27 1.27)) (justify left))
-    (property "Intersheetrefs" "${INTERSHEET_REFS}" (at 202.5602 93.98 0)
+  (global_label "STM32H743_GPIO_EXTI1" (shape bidirectional) (at 177.8 124.46 0) (fields_autoplaced)
+    (effects (font (size 1.27 1.27)) (justify left))
+    (property "Intersheetrefs" "${INTERSHEET_REFS}" (at 204.3745 124.46 0)
       (effects (font (size 1.27 1.27)) (justify left) hide)
     )
@@
     )
   )
+  (global_label "STM32H743_GPIO_OUT_PC0" (shape bidirectional) (at 177.8 121.92 0) (fields_autoplaced)
+    (effects (font (size 1.27 1.27)) (justify left))
+    (property "Intersheetrefs" "${INTERSHEET_REFS}" (at 207.5798 121.92 0)
+      (effects (font (size 1.27 1.27)) (justify left) hide)
+    )
+  )
   (global_label "STM32H743_GPIO_EXTI6" (shape bidirectional) (at 134.62 116.84 180) (fields_autoplaced)
     (effects (font (size 1.27 1.27)) (justify right))
@@
     )
   )
+  (global_label "STM32H743_TIM4_CH1" (shape bidirectional) (at 177.8 93.98 0) (fields_autoplaced)
+    (effects (font (size 1.27 1.27)) (justify left))
+    (property "Intersheetrefs" "${INTERSHEET_REFS}" (at 202.8021 93.98 0)
+      (effects (font (size 1.27 1.27)) (justify left) hide)
+    )
+  )
   (global_label "STM32H743_ADC12_INP3" (shape bidirectional) (at 177.8 50.8 0) (fields_autoplaced)
     (effects (font (size 1.27 1.27)) (justify left))
@@
     )
   )
+  (global_label "STM32H743_I2C1_SCL" (shape bidirectional) (at 177.8 99.06 0) (fields_autoplaced)
+    (effects (font (size 1.27 1.27)) (justify left))
+    (property "Intersheetrefs" "${INTERSHEET_REFS}" (at 202.5602 99.06 0)
+      (effects (font (size 1.27 1.27)) (justify left) hide)
+    )
+  )

Commit message: feat: hardware: Assigns footprints for resistors
Parts:
- R? (x4): footprint (none) -> Resistor_SMD:R_0402_1005Metric
Changed lines of the file:
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@@
       (effects (font (size 1.27 1.27)) (justify left))
     )
-    (property "Footprint" "" (at 88.9 50.8 0)
+    (property "Footprint" "Resistor_SMD:R_0402_1005Metric" (at 88.9 50.8 0)
       (effects (font (size 1.27 1.27)) hide)
     )
@@
       (effects (font (size 1.27 1.27)) (justify right))
     )
-    (property "Footprint" "" (at 99.06 96.52 0)
+    (property "Footprint" "Resistor_SMD:R_0402_1005Metric" (at 99.06 96.52 0)
       (effects (font (size 1.27 1.27)) hide)
     )
@@
       (effects (font (size 1.27 1.27)) (justify right))
     )
-    (property "Footprint" "" (at 88.9 73.66 0)
+    (property "Footprint" "Resistor_SMD:R_0402_1005Metric" (at 88.9 73.66 0)
       (effects (font (size 1.27 1.27)) hide)
     )
@@
       (effects (font (size 1.27 1.27)))
     )
-    (property "Footprint" "" (at 73.66 40.64 0)
-      (effects (font (size 1.27 1.27)) hide)
-    )
+    (property "Footprint" "Resistor_SMD:R_0402_1005Metric" (at 73.66 40.64 0)
+      (effects (font (size 1.27 1.27)) hide)
+    )

Commit message: feat: hardware: Assigns footprints for caps #3
Parts:
- C? (x9): footprint (none) -> Capacitor_SMD:C_0805_2012Metric
- C? (x5): footprint (none) -> Capacitor_SMD:C_1210_3225Metric
Changed lines of the file:
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@@
       (effects (font (size 1.27 1.27)) (justify right))
     )
-    (property "Footprint" "" (at 53.34 25.4 0)
+    (property "Footprint" "Capacitor_SMD:C_0805_2012Metric" (at 53.34 25.4 0)
       (effects (font (size 1.27 1.27)) hide)
     )
@@
       (effects (font (size 1.27 1.27)) (justify right))
     )
-    (property "Footprint" "" (at 63.5 25.4 0)
+    (property "Footprint" "Capacitor_SMD:C_0805_2012Metric" (at 63.5 25.4 0)
       (effects (font (size 1.27 1.27)) hide)
     )
@@
       (effects (font (size 1.27 1.27)) (justify right))
     )
-    (property "Footprint" "" (at 119.38 152.4 0)
+    (property "Footprint" "Capacitor_SMD:C_1210_3225Metric" (at 119.38 152.4 0)
       (effects (font (size 1.27 1.27)) hide)
     )
@@
       (effects (font (size 1.27 1.27)) (justify right))
     )
-    (property "Footprint" "" (at 93.98 25.4 0)
+    (property "Footprint" "Capacitor_SMD:C_0805_2012Metric" (at 93.98 25.4 0)
       (effects (font (size 1.27 1.27)) hide)
     )
@@
       (effects (font (size 1.27 1.27)) (justify right))
     )
-    (property "Footprint" "" (at 43.18 50.8 0)
+    (property "Footprint" "Capacitor_SMD:C_1210_3225Metric" (at 43.18 50.8 0)
       (effects (font (size 1.27 1.27)) hide)
     )
@@
       (effects (font (size 1.27 1.27)) (justify right))
     )
-    (property "Footprint" "" (at 53.34 50.8 0)
+    (property "Footprint" "Capacitor_SMD:C_0805_2012Metric" (at 53.34 50.8 0)
       (effects (font (size 1.27 1.27)) hide)
     )
@@
       (effects (font (size 1.27 1.27)) (justify right))
     )
-    (property "Footprint" "" (at 104.14 25.4 0)
+    (property "Footprint" "Capacitor_SMD:C_0805_2012Metric" (at 104.14 25.4 0)
       (effects (font (size 1.27 1.27)) hide)
     )
@@
       (effects (font (size 1.27 1.27)) (justify right))
     )
-    (property "Footprint" "" (at 113.03 30.48 0)
+    (property "Footprint" "Capacitor_SMD:C_0805_2012Metric" (at 113.03 30.48 0)
       (effects (font (size 1.27 1.27)) hide)
     )
@@
       (effects (font (size 1.27 1.27)) (justify right))
     )
-    (property "Footprint" "" (at 208.28 25.4 0)
+    (property "Footprint" "Capacitor_SMD:C_1210_3225Metric" (at 208.28 25.4 0)
       (effects (font (size 1.27 1.27)) hide)
     )
@@
       (effects (font (size 1.27 1.27)) (justify right))
     )
-    (property "Footprint" "" (at 83.82 25.4 0)
+    (property "Footprint" "Capacitor_SMD:C_0805_2012Metric" (at 83.82 25.4 0)
       (effects (font (size 1.27 1.27)) hide)
     )
@@
       (effects (font (size 1.27 1.27)) (justify right))
     )
-    (property "Footprint" "" (at 198.12 25.4 0)
+    (property "Footprint" "Capacitor_SMD:C_0805_2012Metric" (at 198.12 25.4 0)
       (effects (font (size 1.27 1.27)) hide)
     )
@@
       (effects (font (size 1.27 1.27)) (justify right))
     )
-    (property "Footprint" "" (at 73.66 25.4 0)
+    (property "Footprint" "Capacitor_SMD:C_0805_2012Metric" (at 73.66 25.4 0)
       (effects (font (size 1.27 1.27)) hide)
     )
@@
       (effects (font (size 1.27 1.27)) (justify right))
     )
-    (property "Footprint" "" (at 129.54 152.4 0)
+    (property "Footprint" "Capacitor_SMD:C_1210_3225Metric" (at 129.54 152.4 0)
       (effects (font (size 1.27 1.27)) hide)
     )
@@
       (effects (font (size 1.27 1.27)) (justify right))
     )
-    (property "Footprint" "" (at 43.18 25.4 0)
-      (effects (font (size 1.27 1.27)) hide)
-    )
+    (property "Footprint" "Capacitor_SMD:C_1210_3225Metric" (at 43.18 25.4 0)
+      (effects (font (size 1.27 1.27)) hide)
+    )

Commit message: feat: hardware: Assigns footprints for caps #5
Parts:
- C?: footprint (none) -> Capacitor_SMD:C_1210_3225Metric
Changed lines of the file:
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@@
       (effects (font (size 1.27 1.27)) (justify right))
     )
-    (property "Footprint" "" (at 78.74 50.8 0)
+    (property "Footprint" "Capacitor_SMD:C_1210_3225Metric" (at 78.74 50.8 0)
       (effects (font (size 1.27 1.27)) hide)
     )
