File: hardware/kicad/tinyscope/power_and_charging.kicad_sch (KiCad schematic)
At the start: 45 parts, among them SW2 SW_SPST

Commit message: fix: hardware: Solves electrical rules warnings and errors #9
Parts:
- removed J?: Conn_01x02, symbol Connector_Generic:Conn_01x02
- added J9: Conn_01x03, symbol Connector_Generic:Conn_01x03
Connections:
- net BQ24075_OUT: no longer C?.1, R?.2, R?.2, U?.10 (OUT), U?.11 (OUT)
- net BQ24075_TS: now also J9.2 (Pin_2)
- net DEV_BATT+: now also J9.1 (Pin_1)
- net GND: now also J9.3 (Pin_3)
- new net: C?.1, R?.2, R?.2, U?.10 (OUT), U?.11 (OUT)
Changed lines of the file:
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@@
   (junction (at 238.76 48.26) (diameter 0) (color 0 0 0 0)
-  )
-  (junction (at 119.38 104.14) (diameter 0) (color 0 0 0 0)
   )
   (junction (at 251.46 111.76) (diameter 0) (color 0 0 0 0)
@@
     (stroke (width 0) (type default))
   )
+  (wire (pts (xy 200.66 148.59) (xy 213.36 148.59))
+    (stroke (width 0) (type default))
+  )
   (wire (pts (xy 193.04 63.5) (xy 195.58 63.5))
     (stroke (width 0) (type default))
@@
     (stroke (width 0) (type default))
   )
-  (wire (pts (xy 99.06 104.14) (xy 119.38 104.14))
+  (wire (pts (xy 99.06 104.14) (xy 129.54 104.14))
     (stroke (width 0) (type default))
   )
@@
     (stroke (width 0) (type default))
   )
-  (wire (pts (xy 203.2 147.32) (xy 213.36 147.32))
-    (stroke (width 0) (type default))
-  )
   (wire (pts (xy 88.9 73.66) (xy 88.9 71.12))
     (stroke (width 0) (type default))
@@
     (stroke (width 0) (type default))
   )
-  (wire (pts (xy 119.38 104.14) (xy 129.54 104.14))
-    (stroke (width 0) (type default))
-  )
   (wire (pts (xy 259.08 50.8) (xy 259.08 48.26))
     (stroke (width 0) (type default))
@@
     (stroke (width 0) (type default))
   )
-  (wire (pts (xy 203.2 149.86) (xy 203.2 152.4))
+  (wire (pts (xy 200.66 151.13) (xy 200.66 153.67))
     (stroke (width 0) (type default))
   )
@@
     (stroke (width 0) (type default))
   )
+  (wire (pts (xy 200.66 146.05) (xy 213.36 146.05))
+    (stroke (width 0) (type default))
+  )
   (wire (pts (xy 25.4 96.52) (xy 25.4 106.68))
     (stroke (width 0) (type default))
   )
-  (wire (pts (xy 119.38 93.98) (xy 119.38 104.14))
-    (stroke (width 0) (type default))
-  )
   (wire (pts (xy 269.24 58.42) (xy 269.24 60.96))
     (stroke (width 0) (type default))
@@
     (stroke (width 0) (type default))
   )
-  (wire (pts (xy 213.36 149.86) (xy 203.2 149.86))
-    (stroke (width 0) (type default))
-  )
   (wire (pts (xy 251.46 116.84) (xy 251.46 111.76))
     (stroke (width 0) (type default))
@@
     (stroke (width 0) (type default))
   )
+  (wire (pts (xy 99.06 116.84) (xy 111.76 116.84))
+    (stroke (width 0) (type default))
+  )
   (wire (pts (xy 50.8 109.22) (xy 50.8 134.62))
     (stroke (width 0) (type default))
@@
   )
   (wire (pts (xy 63.5 73.66) (xy 71.12 73.66))
+    (stroke (width 0) (type default))
+  )
+  (wire (pts (xy 200.66 151.13) (xy 213.36 151.13))
     (stroke (width 0) (type default))
   )
@@
     (effects (font (size 1.27 1.27) bold) (justify right bottom))
   )
-  (label "BQ24075_CEB" (at 58.42 109.22 0) (fields_autoplaced)
-    (effects (font (size 1.27 1.27) bold) (justify left bottom))
-  )
-  (label "BQ24075_EN1" (at 58.42 114.3 0) (fields_autoplaced)
-    (effects (font (size 1.27 1.27) bold) (justify left bottom))
+  (label "BQ24075_TS" (at 111.76 116.84 180) (fields_autoplaced)
+    (effects (font (size 1.27 1.27) bold) (justify right bottom))
   )
   (label "EXT_BATT+" (at 160.02 147.32 0) (fields_autoplaced)
@@
     (effects (font (size 1.27 1.27) bold) (justify left bottom))
   )
+  (label "BQ24075_TS" (at 200.66 148.59 0) (fields_autoplaced)
+    (effects (font (size 1.27 1.27) bold) (justify left bottom))
+  )
   (label "DEV_BATT+" (at 58.42 162.56 180) (fields_autoplaced)
     (effects (font (size 1.27 1.27) bold) (justify right bottom))
@@
     (effects (font (size 1.27 1.27) bold) (justify right bottom))
   )
-  (label "DEV_BATT+" (at 203.2 147.32 0) (fields_autoplaced)
+  (label "DEV_BATT+" (at 200.66 146.05 0) (fields_autoplaced)
     (effects (font (size 1.27 1.27) bold) (justify left bottom))
   )
   (label "USBC_VOUT" (at 228.6 106.68 0) (fields_autoplaced)
-    (effects (font (size 1.27 1.27) bold) (justify left bottom))
-  )
-  (label "BQ24075_EN2" (at 58.42 116.84 0) (fields_autoplaced)
     (effects (font (size 1.27 1.27) bold) (justify left bottom))
   )
@@
     (effects (font (size 1.27 1.27)) (justify left))
     (property "Intersheetrefs" "${INTERSHEET_REFS}" (at 132.2871 51.435 0)
-      (effects (font (size 1.27 1.27)) (justify left) hide)
-    )
-  )
-  (global_label "BQ24075_TS" (shape bidirectional) (at 99.06 116.84 0) (fields_autoplaced)
-    (effects (font (size 1.27 1.27)) (justify left))
-    (property "Intersheetrefs" "${INTERSHEET_REFS}" (at 114.8698 116.84 0)
       (effects (font (size 1.27 1.27)) (justify left) hide)
     )
@@
     )
   )
-  (symbol (lib_id "power:GND") (at 203.2 152.4 0) (unit 1)
+  (symbol (lib_id "power:GND") (at 200.66 153.67 0) (unit 1)
     (in_bom yes) (on_board yes) (dnp no) (fields_autoplaced)
-    (property "Reference" "#PWR?" (at 203.2 158.75 0)
-      (effects (font (size 1.27 1.27)) hide)
-    )
-    (property "Value" "GND" (at 203.2 157.48 0)
-      (effects (font (size 1.27 1.27)) hide)
-    )
-    (property "Footprint" "" (at 203.2 152.4 0)
-      (effects (font (size 1.27 1.27)) hide)
-    )
-    (property "Datasheet" "" (at 203.2 152.4 0)
+    (property "Reference" "#PWR?" (at 200.66 160.02 0)
+      (effects (font (size 1.27 1.27)) hide)
+    )
+    (property "Value" "GND" (at 200.66 158.75 0)
+      (effects (font (size 1.27 1.27)) hide)
+    )
+    (property "Footprint" "" (at 200.66 153.67 0)
+      (effects (font (size 1.27 1.27)) hide)
+    )
+    (property "Datasheet" "" (at 200.66 153.67 0)
       (effects (font (size 1.27 1.27)) hide)
     )
@@
     )
   )
-  (symbol (lib_id "Connector_Generic:Conn_01x02") (at 218.44 147.32 0) (unit 1)
-    (in_bom yes) (on_board yes) (dnp no)
-    (property "Reference" "J?" (at 217.17 144.78 0)
-      (effects (font (size 1.27 1.27)) (justify left))
-    )
-    (property "Value" "Conn_01x02" (at 220.98 149.86 0)
-      (effects (font (size 1.27 1.27)) (justify left) hide)
-    )
-    (property "Footprint" "" (at 218.44 147.32 0)
-      (effects (font (size 1.27 1.27)) hide)
-    )
-    (property "Datasheet" "~" (at 218.44 147.32 0)
-      (effects (font (size 1.27 1.27)) hide)
-    )
-    (pin "1")
-    (pin "2")
-    (instances
-      (project "tinyscope"
-        (path "/bb072e32-cc57-415a-8554-0e84d374f333"
-          (reference "J?") (unit 1)
-        )
-        (path "/bb072e32-cc57-415a-8554-0e84d374f333/7c1b1425-60eb-4f71-b125-42ba246f39fb"
-          (reference "J3") (unit 1)
-        )
-      )
-    )
-  )
   (symbol (lib_id "Device:C_Small") (at 25.4 109.22 0) (unit 1)
     (in_bom yes) (on_board yes) (dnp no)
@@
         )
       )
+    )
+  )
+  (symbol (lib_id "Connector_Generic:Conn_01x03") (at 218.44 148.59 0) (unit 1)
+    (in_bom yes) (on_board yes) (dnp no) (fields_autoplaced)
+    (property "Reference" "J9" (at 220.98 147.32 0)
+      (effects (font (size 1.27 1.27)) (justify left))
+    )
+    (property "Value" "Conn_01x03" (at 220.98 149.86 0)
+      (effects (font (size 1.27 1.27)) (justify left))
+    )
+    (property "Footprint" "" (at 218.44 148.59 0)
+      (effects (font (size 1.27 1.27)) hide)
+    )
+    (property "Datasheet" "~" (at 218.44 148.59 0)
+      (effects (font (size 1.27 1.27)) hide)
+    )
+    (pin "1")
+    (pin "2")
+    (pin "3")
+    (instances
+      (project "tinyscope"
+        (path "/bb072e32-cc57-415a-8554-0e84d374f333/7c1b1425-60eb-4f71-b125-42ba246f39fb"
+          (reference "J9") (unit 1)
+        )
+      )

Commit message: feat: hardware: Assigns footprints to USBC part
Parts:
- J?: footprint (none) -> Connector_USB:USB_C_Receptacle_GCT_USB4105-xx-A_16P_TopMnt_Horizontal
- R? (x2): footprint (none) -> Resistor_SMD:R_0402_1005Metric
Changed lines of the file:
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@@
       (effects (font (size 1.27 1.27)) (justify left))
     )
-    (property "Footprint" "" (at 91.44 68.58 0)
+    (property "Footprint" "Resistor_SMD:R_0402_1005Metric" (at 91.44 68.58 0)
       (effects (font (size 1.27 1.27)) hide)
     )
@@
       (effects (font (size 1.27 1.27)) hide)
     )
-    (property "Footprint" "" (at 74.93 48.26 0)
+    (property "Footprint" "Connector_USB:USB_C_Receptacle_GCT_USB4105-xx-A_16P_TopMnt_Horizontal" (at 74.93 48.26 0)
       (effects (font (size 1.27 1.27)) hide)
     )
@@
       (effects (font (size 1.27 1.27)) (justify right))
     )
-    (property "Footprint" "" (at 88.9 68.58 0)
-      (effects (font (size 1.27 1.27)) hide)
-    )
+    (property "Footprint" "Resistor_SMD:R_0402_1005Metric" (at 88.9 68.58 0)
+      (effects (font (size 1.27 1.27)) hide)
+    )

Commit message: feat: hardware: Assigns footprints for resistors
Parts:
- R? (x13): footprint (none) -> Resistor_SMD:R_0402_1005Metric
Changed lines of the file:
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@@
       (effects (font (size 1.27 1.27)) (justify right))
     )
-    (property "Footprint" "" (at 134.62 109.22 0)
+    (property "Footprint" "Resistor_SMD:R_0402_1005Metric" (at 134.62 109.22 0)
       (effects (font (size 1.27 1.27)) hide)
     )
@@
       (effects (font (size 1.27 1.27)) (justify right))
     )
-    (property "Footprint" "" (at 185.42 127 0)
+    (property "Footprint" "Resistor_SMD:R_0402_1005Metric" (at 185.42 127 0)
       (effects (font (size 1.27 1.27)) hide)
     )
@@
       (effects (font (size 1.27 1.27)) (justify right))
     )
-    (property "Footprint" "" (at 177.8 63.5 0)
+    (property "Footprint" "Resistor_SMD:R_0402_1005Metric" (at 177.8 63.5 0)
       (effects (font (size 1.27 1.27)) hide)
     )
@@
       (effects (font (size 1.27 1.27)) (justify right))
     )
-    (property "Footprint" "" (at 177.8 48.26 0)
+    (property "Footprint" "Resistor_SMD:R_0402_1005Metric" (at 177.8 48.26 0)
       (effects (font (size 1.27 1.27)) hide)
     )
@@
       (effects (font (size 1.27 1.27)) (justify right))
     )
-    (property "Footprint" "" (at 142.24 109.22 0)
+    (property "Footprint" "Resistor_SMD:R_0402_1005Metric" (at 142.24 109.22 0)
       (effects (font (size 1.27 1.27)) hide)
     )
@@
       (effects (font (size 1.27 1.27)) (justify left))
     )
-    (property "Footprint" "" (at 38.1 129.54 0)
+    (property "Footprint" "Resistor_SMD:R_0402_1005Metric" (at 38.1 129.54 0)
       (effects (font (size 1.27 1.27)) hide)
     )
@@
       (effects (font (size 1.27 1.27)) (justify left))
     )
-    (property "Footprint" "" (at 269.24 53.34 0)
+    (property "Footprint" "Resistor_SMD:R_0402_1005Metric" (at 269.24 53.34 0)
       (effects (font (size 1.27 1.27)) hide)
     )
@@
       (effects (font (size 1.27 1.27)) (justify left))
     )
-    (property "Footprint" "" (at 269.24 63.5 0)
+    (property "Footprint" "Resistor_SMD:R_0402_1005Metric" (at 269.24 63.5 0)
       (effects (font (size 1.27 1.27)) hide)
     )
@@
       (effects (font (size 1.27 1.27)) (justify left))
     )
-    (property "Footprint" "" (at 182.88 63.5 0)
+    (property "Footprint" "Resistor_SMD:R_0402_1005Metric" (at 182.88 63.5 0)
       (effects (font (size 1.27 1.27)) hide)
     )
@@
       (effects (font (size 1.27 1.27)) (justify right))
     )
-    (property "Footprint" "" (at 226.06 55.88 0)
+    (property "Footprint" "Resistor_SMD:R_0402_1005Metric" (at 226.06 55.88 0)
       (effects (font (size 1.27 1.27)) hide)
     )
@@
       (effects (font (size 1.27 1.27)) (justify right))
     )
-    (property "Footprint" "" (at 33.02 129.54 0)
+    (property "Footprint" "Resistor_SMD:R_0402_1005Metric" (at 33.02 129.54 0)
       (effects (font (size 1.27 1.27)) hide)
     )
@@
       (effects (font (size 1.27 1.27)) (justify left))
     )
-    (property "Footprint" "" (at 71.12 129.54 0)
+    (property "Footprint" "Resistor_SMD:R_0402_1005Metric" (at 71.12 129.54 0)
       (effects (font (size 1.27 1.27)) hide)
     )
@@
       (effects (font (size 1.27 1.27)) (justify left))
     )
-    (property "Footprint" "" (at 63.5 129.54 0)
-      (effects (font (size 1.27 1.27)) hide)
-    )
+    (property "Footprint" "Resistor_SMD:R_0402_1005Metric" (at 63.5 129.54 0)
+      (effects (font (size 1.27 1.27)) hide)
+    )
