File: hardware/kicad/tinyscope/power_and_charging.kicad_sch (KiCad schematic)
At the start: 45 parts, among them J9 Conn_01x03, SW2 SW_SPST

Commit message: feat: hardware: Assigns footprints for TPS63802DLAR voltage regulator and MAX17048 fuel gauge
Parts:
- U?: footprint SON50P200X200X80-9N-D -> Package_SON:SON50P200X200X80-9N-D
Changed lines of the file:
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@@
       (effects (font (size 1.27 1.27)))
     )
-    (property "Footprint" "SON50P200X200X80-9N-D" (at 85.09 254.94 0)
+    (property "Footprint" "Package_SON:SON50P200X200X80-9N-D" (at 85.09 254.94 0)
       (effects (font (size 1.27 1.27)) (justify left top) hide)
     )

Commit message: feat: hardware: Assigns footprints for caps #1
Parts:
- C? (x2): footprint (none) -> Capacitor_SMD:C_1210_3225Metric
Changed lines of the file:
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@@
       (effects (font (size 1.27 1.27)) (justify right))
     )
-    (property "Footprint" "" (at 167.64 48.26 0)
+    (property "Footprint" "Capacitor_SMD:C_1210_3225Metric" (at 167.64 48.26 0)
       (effects (font (size 1.27 1.27)) hide)
     )
@@
       (effects (font (size 1.27 1.27)) (justify right))
     )
-    (property "Footprint" "" (at 157.48 48.26 0)
-      (effects (font (size 1.27 1.27)) hide)
-    )
+    (property "Footprint" "Capacitor_SMD:C_1210_3225Metric" (at 157.48 48.26 0)
+      (effects (font (size 1.27 1.27)) hide)
+    )

Commit message: feat: hardware: Assigns footprints for caps #2
Parts:
- C? (x3): footprint (none) -> Capacitor_SMD:C_1210_3225Metric
- C? (x2): footprint (none) -> Capacitor_THT:C_Radial_D6.3mm_H5.0mm_P2.50mm
Changed lines of the file:
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@@
       (effects (font (size 1.27 1.27)) (justify right))
     )
-    (property "Footprint" "" (at 236.22 63.5 0)
+    (property "Footprint" "Capacitor_SMD:C_1210_3225Metric" (at 236.22 63.5 0)
       (effects (font (size 1.27 1.27)) hide)
     )
@@
       (effects (font (size 1.27 1.27)) (justify right))
     )
-    (property "Footprint" "" (at 218.44 116.84 0)
+    (property "Footprint" "Capacitor_SMD:C_1210_3225Metric" (at 218.44 116.84 0)
       (effects (font (size 1.27 1.27)) hide)
     )
@@
       (effects (font (size 1.27 1.27)) (justify left))
     )
-    (property "Footprint" "" (at 259.08 53.34 0)
+    (property "Footprint" "Capacitor_THT:C_Radial_D6.3mm_H5.0mm_P2.50mm" (at 259.08 53.34 0)
       (effects (font (size 1.27 1.27)) hide)
     )
@@
       (effects (font (size 1.27 1.27)) (justify right))
     )
-    (property "Footprint" "" (at 226.06 63.5 0)
+    (property "Footprint" "Capacitor_SMD:C_1210_3225Metric" (at 226.06 63.5 0)
       (effects (font (size 1.27 1.27)) hide)
     )
@@
       (effects (font (size 1.27 1.27)) (justify left))
     )
-    (property "Footprint" "" (at 248.92 53.34 0)
-      (effects (font (size 1.27 1.27)) hide)
-    )
-    (property "Datasheet" "~" (at 248.92 53.34 0)
-      (effects (font (size 1.27 1.27)) hide)
-    )
+    (property "Footprint" "Capacitor_THT:C_Radial_D6.3mm_H5.0mm_P2.50mm" (at 248.92 53.34 0)
+      (effects (font (size 1.27 1.27)) hide)
+    )
+    (property "Datasheet" "https://www.we-online.com/components/products/datasheet/860020673013.pdf" (at 248.92 53.34 0)
+      (effects (font (size 1.27 1.27)) hide)
+    )

Commit message: feat: hardware: Assigns footprints for caps #3
Parts:
- C? (x2): footprint (none) -> Capacitor_SMD:C_0805_2012Metric
- C? (x3): footprint (none) -> Capacitor_SMD:C_1210_3225Metric
Changed lines of the file:
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@@
       (effects (font (size 1.27 1.27)))
     )
-    (property "Footprint" "" (at 215.9 43.18 0)
+    (property "Footprint" "Capacitor_SMD:C_0805_2012Metric" (at 215.9 43.18 0)
       (effects (font (size 1.27 1.27)) hide)
     )
@@
       (effects (font (size 1.27 1.27)) (justify right))
     )
-    (property "Footprint" "" (at 119.38 116.84 0)
+    (property "Footprint" "Capacitor_SMD:C_1210_3225Metric" (at 119.38 116.84 0)
       (effects (font (size 1.27 1.27)) hide)
     )
@@
       (effects (font (size 1.27 1.27)) (justify right))
     )
-    (property "Footprint" "" (at 43.18 170.18 0)
+    (property "Footprint" "Capacitor_SMD:C_0805_2012Metric" (at 43.18 170.18 0)
       (effects (font (size 1.27 1.27)) hide)
     )
@@
       (effects (font (size 1.27 1.27)) (justify right))
     )
-    (property "Footprint" "" (at 25.4 109.22 0)
+    (property "Footprint" "Capacitor_SMD:C_1210_3225Metric" (at 25.4 109.22 0)
       (effects (font (size 1.27 1.27)) hide)
     )
@@
       (effects (font (size 1.27 1.27)) (justify right))
     )
-    (property "Footprint" "" (at 129.54 116.84 0)
-      (effects (font (size 1.27 1.27)) hide)
-    )
+    (property "Footprint" "Capacitor_SMD:C_1210_3225Metric" (at 129.54 116.84 0)
+      (effects (font (size 1.27 1.27)) hide)
+    )

Commit message: feat: hardware: Assigns footprints for caps #4
Parts:
- C?: footprint Capacitor_SMD:C_1210_3225Metric -> Capacitor_SMD:C_0603_1608Metric
- C?: footprint Capacitor_SMD:C_1210_3225Metric -> Capacitor_SMD:C_0805_2012Metric
Changed lines of the file:
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@@
       (effects (font (size 1.27 1.27)) (justify right))
     )
-    (property "Footprint" "Capacitor_SMD:C_1210_3225Metric" (at 218.44 116.84 0)
+    (property "Footprint" "Capacitor_SMD:C_0603_1608Metric" (at 218.44 116.84 0)
       (effects (font (size 1.27 1.27)) hide)
     )
@@
       (effects (font (size 1.27 1.27)) (justify right))
     )
-    (property "Footprint" "Capacitor_SMD:C_1210_3225Metric" (at 157.48 48.26 0)
-      (effects (font (size 1.27 1.27)) hide)
-    )
+    (property "Footprint" "Capacitor_SMD:C_0805_2012Metric" (at 157.48 48.26 0)
+      (effects (font (size 1.27 1.27)) hide)
+    )

Commit message: feat: hardware: Assigns footprints for caps #5
Parts:
- C?: footprint Capacitor_SMD:C_0805_2012Metric -> Capacitor_SMD:C_0603_1608Metric
- C?: footprint Capacitor_SMD:C_1210_3225Metric -> Capacitor_SMD:C_0805_2012Metric
- C?: footprint Capacitor_SMD:C_0805_2012Metric -> Capacitor_SMD:C_1210_3225Metric
- C?: footprint Capacitor_SMD:C_1210_3225Metric -> Capacitor_SMD:C_0603_1608Metric
- D?: footprint (none) -> Diode_SMD:D_SOD-323
- F?: footprint (none) -> Fuse:Fuse_0805_2012Metric
Changed lines of the file:
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@@
       (effects (font (size 1.27 1.27)))
     )
-    (property "Footprint" "Capacitor_SMD:C_0805_2012Metric" (at 215.9 43.18 0)
-      (effects (font (size 1.27 1.27)) hide)
-    )
-    (property "Datasheet" "~" (at 215.9 43.18 0)
+    (property "Footprint" "Capacitor_SMD:C_0603_1608Metric" (at 215.9 43.18 0)
+      (effects (font (size 1.27 1.27)) hide)
+    )
+    (property "Datasheet" "https://www.mouser.pl/en/ProductDetail/Murata-Electronics/GCM188R71H104KA57D?qs=aEuGZpxfbxWuy5eQGqiN%252BA%3D%3D" (at 215.9 43.18 0)
       (effects (font (size 1.27 1.27)) hide)
     )
@@
       (effects (font (size 1.27 1.27)) (justify right))
     )
-    (property "Footprint" "Capacitor_SMD:C_1210_3225Metric" (at 236.22 63.5 0)
-      (effects (font (size 1.27 1.27)) hide)
-    )
-    (property "Datasheet" "~" (at 236.22 63.5 0)
+    (property "Footprint" "Capacitor_SMD:C_0805_2012Metric" (at 236.22 63.5 0)
+      (effects (font (size 1.27 1.27)) hide)
+    )
+    (property "Datasheet" "https://www.mouser.pl/en/ProductDetail/KEMET/C0805C390K1RACTU?qs=sGAEpiMZZMt7gvpyg0xT8tCg5CynaY7NQtUIV8TPugXj3aQJYHS6Rw%3D%3D" (at 236.22 63.5 0)
       (effects (font (size 1.27 1.27)) hide)
     )
@@
       (effects (font (size 1.27 1.27)) hide)
     )
-    (property "Datasheet" "~" (at 167.64 48.26 0)
+    (property "Datasheet" "https://www.mouser.pl/en/ProductDetail/KYOCERA-AVX/KGM32LR72A225KL?qs=sGAEpiMZZMuMW9TJLBQkXqLYvz3DzaXfhkDBFYHfN0A%3D" (at 167.64 48.26 0)
       (effects (font (size 1.27 1.27)) hide)
     )
@@
       (effects (font (size 1.27 1.27)) (justify right))
     )
-    (property "Footprint" "Capacitor_SMD:C_0805_2012Metric" (at 157.48 48.26 0)
-      (effects (font (size 1.27 1.27)) hide)
-    )
-    (property "Datasheet" "~" (at 157.48 48.26 0)
+    (property "Footprint" "Capacitor_SMD:C_1210_3225Metric" (at 157.48 48.26 0)
+      (effects (font (size 1.27 1.27)) hide)
+    )
+    (property "Datasheet" "https://www.mouser.pl/en/ProductDetail/KYOCERA-AVX/KGM32LR72A225KL?qs=sGAEpiMZZMuMW9TJLBQkXqLYvz3DzaXfhkDBFYHfN0A%3D" (at 157.48 48.26 0)
       (effects (font (size 1.27 1.27)) hide)
     )
@@
       (effects (font (size 1.27 1.27)) (justify left))
     )
-    (property "Footprint" "" (at 193.04 116.84 90)
-      (effects (font (size 1.27 1.27)) hide)
-    )
-    (property "Datasheet" "~" (at 193.04 116.84 90)
+    (property "Footprint" "Diode_SMD:D_SOD-323" (at 193.04 116.84 90)
+      (effects (font (size 1.27 1.27)) hide)
+    )
+    (property "Datasheet" "https://www.mouser.pl/en/ProductDetail/Vishay/BZX384C15-HE3_A08?qs=CoAU%2FpHVZXxvC6kVCkxPeg%3D%3D" (at 193.04 116.84 90)
       (effects (font (size 1.27 1.27)) hide)
     )
@@
       (effects (font (size 1.27 1.27)) (justify right))
     )
-    (property "Footprint" "Capacitor_SMD:C_1210_3225Metric" (at 226.06 63.5 0)
-      (effects (font (size 1.27 1.27)) hide)
-    )
-    (property "Datasheet" "~" (at 226.06 63.5 0)
+    (property "Footprint" "Capacitor_SMD:C_0603_1608Metric" (at 226.06 63.5 0)
+      (effects (font (size 1.27 1.27)) hide)
+    )
+    (property "Datasheet" "https://www.mouser.pl/en/ProductDetail/KYOCERA-AVX/KAM15AR72A682KT?qs=sGAEpiMZZMt7gvpyg0xT8jBHDtGZvLzXmmWlq109%252BuwnEcrf4iGzXw%3D%3D" (at 226.06 63.5 0)
       (effects (font (size 1.27 1.27)) hide)
     )
@@
       (effects (font (size 1.27 1.27)))
     )
-    (property "Footprint" "" (at 175.26 111.76 0)
-      (effects (font (size 1.27 1.27)) hide)
-    )
-    (property "Datasheet" "~" (at 175.26 111.76 0)
-      (effects (font (size 1.27 1.27)) hide)
-    )
+    (property "Footprint" "Fuse:Fuse_0805_2012Metric" (at 175.26 111.76 0)
+      (effects (font (size 1.27 1.27)) hide)
+    )
+    (property "Datasheet" "https://www.mouser.pl/en/ProductDetail/Kamaya/FCC20202AATP?qs=sGAEpiMZZMsIz3CjQ1xegZx2pdJYlyprNnQN9Ug27dAO3nKjMfGrww%3D%3D" (at 175.26 111.76 0)
+      (effects (font (size 1.27 1.27)) hide)
+    )

Commit message: feat: hardware: Assigns footprints for connectors #1
Parts:
- J9: footprint (none) -> Connector_PinHeader_2.54mm:PinHeader_1x03_P2.54mm_Vertical_SMD_Pin1Left
- J?: footprint (none) -> Connector_PinHeader_2.54mm:PinHeader_1x02_P2.54mm_Vertical_SMD_Pin1Left
Changed lines of the file:
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@@
       (effects (font (size 1.27 1.27)) (justify left) hide)
     )
-    (property "Footprint" "" (at 175.26 147.32 0)
+    (property "Footprint" "Connector_PinHeader_2.54mm:PinHeader_1x02_P2.54mm_Vertical_SMD_Pin1Left" (at 175.26 147.32 0)
       (effects (font (size 1.27 1.27)) hide)
     )
@@
       (effects (font (size 1.27 1.27)) (justify left))
     )
-    (property "Footprint" "" (at 218.44 148.59 0)
-      (effects (font (size 1.27 1.27)) hide)
-    )
+    (property "Footprint" "Connector_PinHeader_2.54mm:PinHeader_1x03_P2.54mm_Vertical_SMD_Pin1Left" (at 218.44 148.59 0)
+      (effects (font (size 1.27 1.27)) hide)
+    )

Commit message: feat: hardware: Assigns footprints for diodes #1
Parts:
- D? (x2): footprint (none) -> Diode_SMD:D_SOD-323
Connections:
- net BQ24075_OUT: now also C?.1, R?.2, R?.2, U?.10 (OUT), U?.11 (OUT)
Other:
- note removed: "The I2C connection is missing."
Changed lines of the file:
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@@
   (junction (at 248.92 48.26) (diameter 0) (color 0 0 0 0)
   )
+  (junction (at 119.38 93.98) (diameter 0) (color 0 0 0 0)
+  )
   (junction (at 269.24 58.42) (diameter 0) (color 0 0 0 0)
   )
@@
   )
   (junction (at 38.1 134.62) (diameter 0) (color 0 0 0 0)
+  )
+  (junction (at 119.38 104.14) (diameter 0) (color 0 0 0 0)
   )
   (no_connect (at 86.36 60.96))
@@
     (stroke (width 0) (type default))
   )
-  (wire (pts (xy 99.06 104.14) (xy 129.54 104.14))
+  (wire (pts (xy 99.06 104.14) (xy 119.38 104.14))
     (stroke (width 0) (type default))
   )
@@
     (stroke (width 0) (type default))
   )
+  (wire (pts (xy 119.38 93.98) (xy 127 93.98))
+    (stroke (width 0) (type default))
+  )
   (wire (pts (xy 185.42 121.92) (xy 185.42 124.46))
     (stroke (width 0) (type default))
@@
     (stroke (width 0) (type default))
   )
+  (wire (pts (xy 119.38 104.14) (xy 129.54 104.14))
+    (stroke (width 0) (type default))
+  )
   (wire (pts (xy 109.22 39.37) (xy 109.22 33.02))
     (stroke (width 0) (type default))
@@
   )
   (wire (pts (xy 86.36 33.02) (xy 109.22 33.02))
+    (stroke (width 0) (type default))
+  )
+  (wire (pts (xy 119.38 93.98) (xy 119.38 104.14))
     (stroke (width 0) (type default))
   )
@@
   (text "Power Input & Charging" (at 20.32 20.32 0)
     (effects (font (size 4 4) (thickness 0.254) bold (color 0 0 0 1)) (justify left bottom))
-  )
-  (text "The I2C connection is missing." (at 114.3 157.48 0)
-    (effects (font (size 1.27 1.27)) (justify left bottom))
   )
   (label "TPS54360_VOUT" (at 228.6 116.84 0) (fields_autoplaced)
@@
     )
   )
-  (global_label "BQ24075_OUT" (shape bidirectional) (at 119.38 93.98 0) (fields_autoplaced)
+  (global_label "BQ24075_OUT" (shape bidirectional) (at 127 93.98 0) (fields_autoplaced)
     (effects (font (size 1.27 1.27)) (justify left))
-    (property "Intersheetrefs" "${INTERSHEET_REFS}" (at 136.6413 93.98 0)
+    (property "Intersheetrefs" "${INTERSHEET_REFS}" (at 144.2613 93.98 0)
       (effects (font (size 1.27 1.27)) (justify left) hide)
     )
@@
       (effects (font (size 1.27 1.27)) (justify right))
     )
-    (property "Footprint" "" (at 246.38 106.68 90)
-      (effects (font (size 1.27 1.27)) hide)
-    )
-    (property "Datasheet" "~" (at 246.38 106.68 90)
+    (property "Footprint" "Diode_SMD:D_SOD-323" (at 246.38 106.68 90)
+      (effects (font (size 1.27 1.27)) hide)
+    )
+    (property "Datasheet" "https://www.mouser.pl/en/ProductDetail/Infineon-Technologies/BAT60AE6327HTSA1?qs=OwbwYO03UsIW3Y2lCXbs8Q%3D%3D" (at 246.38 106.68 90)
       (effects (font (size 1.27 1.27)) hide)
     )
@@
       (effects (font (size 1.27 1.27)) (justify right))
     )
-    (property "Footprint" "" (at 246.38 116.84 90)
-      (effects (font (size 1.27 1.27)) hide)
-    )
-    (property "Datasheet" "~" (at 246.38 116.84 90)
-      (effects (font (size 1.27 1.27)) hide)
-    )
+    (property "Footprint" "Diode_SMD:D_SOD-323" (at 246.38 116.84 90)
+      (effects (font (size 1.27 1.27)) hide)
+    )
+    (property "Datasheet" "https://www.mouser.pl/en/ProductDetail/Infineon-Technologies/BAT60AE6327HTSA1?qs=OwbwYO03UsIW3Y2lCXbs8Q%3D%3D" (at 246.38 116.84 90)
+      (effects (font (size 1.27 1.27)) hide)
+    )
