File: hardware/kicad/tinyscope/front_end.kicad_sch (KiCad schematic)
At the start: 37 parts, among them J6 Front End A, J7 Front End B, U13 AD8066ARZ-RL, U14 AD8066ARZ-RL, U15 AD8066ARZ-RL

Commit message: feat: hardware: Assigns footprints for resistors
Parts:
- R? (x16): footprint (none) -> Resistor_SMD:R_0402_1005Metric
Changed lines of the file:
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@@
       (effects (font (size 1.27 1.27)))
     )
-    (property "Footprint" "" (at 63.5 126.365 0)
+    (property "Footprint" "Resistor_SMD:R_0402_1005Metric" (at 63.5 126.365 0)
       (effects (font (size 1.27 1.27)) hide)
     )
@@
       (effects (font (size 1.27 1.27)) (justify left))
     )
-    (property "Footprint" "" (at 130.81 71.755 0)
+    (property "Footprint" "Resistor_SMD:R_0402_1005Metric" (at 130.81 71.755 0)
       (effects (font (size 1.27 1.27)) hide)
     )
@@
       (effects (font (size 1.27 1.27)))
     )
-    (property "Footprint" "" (at 175.26 59.055 0)
+    (property "Footprint" "Resistor_SMD:R_0402_1005Metric" (at 175.26 59.055 0)
       (effects (font (size 1.27 1.27)) hide)
     )
@@
       (effects (font (size 1.27 1.27)) (justify left))
     )
-    (property "Footprint" "" (at 130.81 135.255 0)
+    (property "Footprint" "Resistor_SMD:R_0402_1005Metric" (at 130.81 135.255 0)
       (effects (font (size 1.27 1.27)) hide)
     )
@@
       (effects (font (size 1.27 1.27)) (justify left))
     )
-    (property "Footprint" "" (at 40.64 66.675 0)
+    (property "Footprint" "Resistor_SMD:R_0402_1005Metric" (at 40.64 66.675 0)
       (effects (font (size 1.27 1.27)) hide)
     )
@@
       (effects (font (size 1.27 1.27)))
     )
-    (property "Footprint" "" (at 144.78 70.485 0)
+    (property "Footprint" "Resistor_SMD:R_0402_1005Metric" (at 144.78 70.485 0)
       (effects (font (size 1.27 1.27)) hide)
     )
@@
       (effects (font (size 1.27 1.27)))
     )
-    (property "Footprint" "" (at 185.42 59.055 0)
+    (property "Footprint" "Resistor_SMD:R_0402_1005Metric" (at 185.42 59.055 0)
       (effects (font (size 1.27 1.27)) hide)
     )
@@
       (effects (font (size 1.27 1.27)))
     )
-    (property "Footprint" "" (at 63.5 61.595 0)
+    (property "Footprint" "Resistor_SMD:R_0402_1005Metric" (at 63.5 61.595 0)
       (effects (font (size 1.27 1.27)) hide)
     )
@@
       (effects (font (size 1.27 1.27)))
     )
-    (property "Footprint" "" (at 144.78 126.365 0)
+    (property "Footprint" "Resistor_SMD:R_0402_1005Metric" (at 144.78 126.365 0)
       (effects (font (size 1.27 1.27)) hide)
     )
@@
       (effects (font (size 1.27 1.27)))
     )
-    (property "Footprint" "" (at 175.26 122.555 0)
+    (property "Footprint" "Resistor_SMD:R_0402_1005Metric" (at 175.26 122.555 0)
       (effects (font (size 1.27 1.27)) hide)
     )
@@
       (effects (font (size 1.27 1.27)) (justify left))
     )
-    (property "Footprint" "" (at 40.64 131.445 0)
+    (property "Footprint" "Resistor_SMD:R_0402_1005Metric" (at 40.64 131.445 0)
       (effects (font (size 1.27 1.27)) hide)
     )
@@
       (effects (font (size 1.27 1.27)))
     )
-    (property "Footprint" "" (at 185.42 122.555 0)
+    (property "Footprint" "Resistor_SMD:R_0402_1005Metric" (at 185.42 122.555 0)
       (effects (font (size 1.27 1.27)) hide)
     )
@@
       (effects (font (size 1.27 1.27)) (justify left))
     )
-    (property "Footprint" "" (at 130.81 79.375 0)
+    (property "Footprint" "Resistor_SMD:R_0402_1005Metric" (at 130.81 79.375 0)
       (effects (font (size 1.27 1.27)) hide)
     )
@@
       (effects (font (size 1.27 1.27)))
     )
-    (property "Footprint" "" (at 144.78 133.985 0)
+    (property "Footprint" "Resistor_SMD:R_0402_1005Metric" (at 144.78 133.985 0)
       (effects (font (size 1.27 1.27)) hide)
     )
@@
       (effects (font (size 1.27 1.27)))
     )
-    (property "Footprint" "" (at 144.78 62.865 0)
+    (property "Footprint" "Resistor_SMD:R_0402_1005Metric" (at 144.78 62.865 0)
       (effects (font (size 1.27 1.27)) hide)
     )
@@
       (effects (font (size 1.27 1.27)) (justify left))
     )
-    (property "Footprint" "" (at 130.81 142.875 0)
-      (effects (font (size 1.27 1.27)) hide)
-    )
+    (property "Footprint" "Resistor_SMD:R_0402_1005Metric" (at 130.81 142.875 0)
+      (effects (font (size 1.27 1.27)) hide)
+    )

Commit message: feat: hardware: Assigns footprints for AD8066ARZ op amp and encoders
Parts:
- U13, U14, U15: footprint SOIC127P600X175-8N -> Package_SO:SOIC127P600X175-8N
Changed lines of the file:
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@@
       (effects (font (size 1.27 1.27)))
     )
-    (property "Footprint" "SOIC127P600X175-8N" (at 233.68 176.835 0)
+    (property "Footprint" "Package_SO:SOIC127P600X175-8N" (at 233.68 176.835 0)
       (effects (font (size 1.27 1.27)) (justify left top) hide)
     )
@@
       (effects (font (size 1.27 1.27)))
     )
-    (property "Footprint" "SOIC127P600X175-8N" (at 121.92 217.475 0)
+    (property "Footprint" "Package_SO:SOIC127P600X175-8N" (at 121.92 217.475 0)
       (effects (font (size 1.27 1.27)) (justify left top) hide)
     )
@@
       (effects (font (size 1.27 1.27)))
     )
-    (property "Footprint" "SOIC127P600X175-8N" (at 121.92 153.975 0)
-      (effects (font (size 1.27 1.27)) (justify left top) hide)
-    )
+    (property "Footprint" "Package_SO:SOIC127P600X175-8N" (at 121.92 153.975 0)
+      (effects (font (size 1.27 1.27)) (justify left top) hide)
+    )

Commit message: feat: hardware: Assigns footprints for caps #3
Parts:
- C? (x4): footprint (none) -> Capacitor_SMD:C_1210_3225Metric
- C? (x3): footprint (none) -> Capacitor_SMD:C_0805_2012Metric
Changed lines of the file:
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@@
       (effects (font (size 1.27 1.27)))
     )
-    (property "Footprint" "" (at 133.35 34.29 0)
+    (property "Footprint" "Capacitor_SMD:C_1210_3225Metric" (at 133.35 34.29 0)
       (effects (font (size 1.27 1.27)) hide)
     )
@@
       (effects (font (size 1.27 1.27)))
     )
-    (property "Footprint" "" (at 97.79 74.295 0)
+    (property "Footprint" "Capacitor_SMD:C_1210_3225Metric" (at 97.79 74.295 0)
       (effects (font (size 1.27 1.27)) hide)
     )
@@
       (effects (font (size 1.27 1.27)))
     )
-    (property "Footprint" "" (at 97.79 147.955 0)
+    (property "Footprint" "Capacitor_SMD:C_0805_2012Metric" (at 97.79 147.955 0)
       (effects (font (size 1.27 1.27)) hide)
     )
@@
       (effects (font (size 1.27 1.27)))
     )
-    (property "Footprint" "" (at 97.79 84.455 0)
+    (property "Footprint" "Capacitor_SMD:C_0805_2012Metric" (at 97.79 84.455 0)
       (effects (font (size 1.27 1.27)) hide)
     )
@@
       (effects (font (size 1.27 1.27)))
     )
-    (property "Footprint" "" (at 133.35 97.79 0)
+    (property "Footprint" "Capacitor_SMD:C_1210_3225Metric" (at 133.35 97.79 0)
       (effects (font (size 1.27 1.27)) hide)
     )
@@
       (effects (font (size 1.27 1.27)))
     )
-    (property "Footprint" "" (at 133.35 107.95 0)
+    (property "Footprint" "Capacitor_SMD:C_0805_2012Metric" (at 133.35 107.95 0)
       (effects (font (size 1.27 1.27)) hide)
     )
@@
       (effects (font (size 1.27 1.27)))
     )
-    (property "Footprint" "" (at 97.79 137.795 0)
-      (effects (font (size 1.27 1.27)) hide)
-    )
+    (property "Footprint" "Capacitor_SMD:C_1210_3225Metric" (at 97.79 137.795 0)
+      (effects (font (size 1.27 1.27)) hide)
+    )
