File: hardware/kicad/tinyscope/hmi.kicad_sch (KiCad schematic)
At the start: 61 parts, among them J8 Waveshare 16498

Commit message: feat: hardware: Assigns footprints for resistors
Parts:
- R? (x36): footprint (none) -> Resistor_SMD:R_0402_1005Metric
Changed lines of the file:
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@@
       (effects (font (size 1.27 1.27)) (justify left))
     )
-    (property "Footprint" "" (at 129.54 55.88 0)
+    (property "Footprint" "Resistor_SMD:R_0402_1005Metric" (at 129.54 55.88 0)
       (effects (font (size 1.27 1.27)) hide)
     )
@@
       (effects (font (size 1.27 1.27)))
     )
-    (property "Footprint" "" (at 30.48 60.96 0)
+    (property "Footprint" "Resistor_SMD:R_0402_1005Metric" (at 30.48 60.96 0)
       (effects (font (size 1.27 1.27)) hide)
     )
@@
       (effects (font (size 1.27 1.27)) (justify right))
     )
-    (property "Footprint" "" (at 223.52 25.4 0)
+    (property "Footprint" "Resistor_SMD:R_0402_1005Metric" (at 223.52 25.4 0)
       (effects (font (size 1.27 1.27)) hide)
     )
@@
       (effects (font (size 1.27 1.27)) (justify right))
     )
-    (property "Footprint" "" (at 165.1 55.88 0)
+    (property "Footprint" "Resistor_SMD:R_0402_1005Metric" (at 165.1 55.88 0)
       (effects (font (size 1.27 1.27)) hide)
     )
@@
       (effects (font (size 1.27 1.27)))
     )
-    (property "Footprint" "" (at 76.2 60.96 0)
+    (property "Footprint" "Resistor_SMD:R_0402_1005Metric" (at 76.2 60.96 0)
       (effects (font (size 1.27 1.27)) hide)
     )
@@
       (effects (font (size 1.27 1.27)))
     )
-    (property "Footprint" "" (at 264.16 119.38 0)
+    (property "Footprint" "Resistor_SMD:R_0402_1005Metric" (at 264.16 119.38 0)
       (effects (font (size 1.27 1.27)) hide)
     )
@@
       (effects (font (size 1.27 1.27)))
     )
-    (property "Footprint" "" (at 264.16 60.96 0)
+    (property "Footprint" "Resistor_SMD:R_0402_1005Metric" (at 264.16 60.96 0)
       (effects (font (size 1.27 1.27)) hide)
     )
@@
       (effects (font (size 1.27 1.27)) (justify right))
     )
-    (property "Footprint" "" (at 71.12 55.88 0)
+    (property "Footprint" "Resistor_SMD:R_0402_1005Metric" (at 71.12 55.88 0)
       (effects (font (size 1.27 1.27)) hide)
     )
@@
       (effects (font (size 1.27 1.27)))
     )
-    (property "Footprint" "" (at 30.48 30.48 0)
+    (property "Footprint" "Resistor_SMD:R_0402_1005Metric" (at 30.48 30.48 0)
       (effects (font (size 1.27 1.27)) hide)
     )
@@
       (effects (font (size 1.27 1.27)) (justify right))
     )
-    (property "Footprint" "" (at 259.08 55.88 0)
+    (property "Footprint" "Resistor_SMD:R_0402_1005Metric" (at 259.08 55.88 0)
       (effects (font (size 1.27 1.27)) hide)
     )
@@
       (effects (font (size 1.27 1.27)) (justify left))
     )
-    (property "Footprint" "" (at 129.54 114.3 0)
+    (property "Footprint" "Resistor_SMD:R_0402_1005Metric" (at 129.54 114.3 0)
       (effects (font (size 1.27 1.27)) hide)
     )
@@
       (effects (font (size 1.27 1.27)))
     )
-    (property "Footprint" "" (at 76.2 119.38 0)
+    (property "Footprint" "Resistor_SMD:R_0402_1005Metric" (at 76.2 119.38 0)
       (effects (font (size 1.27 1.27)) hide)
     )
@@
       (effects (font (size 1.27 1.27)) (justify right))
     )
-    (property "Footprint" "" (at 71.12 114.3 0)
+    (property "Footprint" "Resistor_SMD:R_0402_1005Metric" (at 71.12 114.3 0)
       (effects (font (size 1.27 1.27)) hide)
     )
@@
       (effects (font (size 1.27 1.27)))
     )
-    (property "Footprint" "" (at 218.44 30.48 0)
+    (property "Footprint" "Resistor_SMD:R_0402_1005Metric" (at 218.44 30.48 0)
       (effects (font (size 1.27 1.27)) hide)
     )
@@
       (effects (font (size 1.27 1.27)) (justify left))
     )
-    (property "Footprint" "" (at 35.56 83.82 0)
+    (property "Footprint" "Resistor_SMD:R_0402_1005Metric" (at 35.56 83.82 0)
       (effects (font (size 1.27 1.27)) hide)
     )
@@
       (effects (font (size 1.27 1.27)))
     )
-    (property "Footprint" "" (at 30.48 88.9 0)
+    (property "Footprint" "Resistor_SMD:R_0402_1005Metric" (at 30.48 88.9 0)
       (effects (font (size 1.27 1.27)) hide)
     )
@@
       (effects (font (size 1.27 1.27)))
     )
-    (property "Footprint" "" (at 170.18 119.38 0)
+    (property "Footprint" "Resistor_SMD:R_0402_1005Metric" (at 170.18 119.38 0)
       (effects (font (size 1.27 1.27)) hide)
     )
@@
       (effects (font (size 1.27 1.27)))
     )
-    (property "Footprint" "" (at 218.44 60.96 0)
+    (property "Footprint" "Resistor_SMD:R_0402_1005Metric" (at 218.44 60.96 0)
       (effects (font (size 1.27 1.27)) hide)
     )
@@
       (effects (font (size 1.27 1.27)) (justify left))
     )
-    (property "Footprint" "" (at 223.52 55.88 0)
+    (property "Footprint" "Resistor_SMD:R_0402_1005Metric" (at 223.52 55.88 0)
       (effects (font (size 1.27 1.27)) hide)
     )
@@
       (effects (font (size 1.27 1.27)) (justify left))
     )
-    (property "Footprint" "" (at 35.56 114.3 0)
+    (property "Footprint" "Resistor_SMD:R_0402_1005Metric" (at 35.56 114.3 0)
       (effects (font (size 1.27 1.27)) hide)
     )
@@
       (effects (font (size 1.27 1.27)) (justify right))
     )
-    (property "Footprint" "" (at 165.1 114.3 0)
+    (property "Footprint" "Resistor_SMD:R_0402_1005Metric" (at 165.1 114.3 0)
       (effects (font (size 1.27 1.27)) hide)
     )
@@
       (effects (font (size 1.27 1.27)) (justify left))
     )
-    (property "Footprint" "" (at 129.54 25.4 0)
+    (property "Footprint" "Resistor_SMD:R_0402_1005Metric" (at 129.54 25.4 0)
       (effects (font (size 1.27 1.27)) hide)
     )
@@
       (effects (font (size 1.27 1.27)))
     )
-    (property "Footprint" "" (at 124.46 30.48 0)
+    (property "Footprint" "Resistor_SMD:R_0402_1005Metric" (at 124.46 30.48 0)
       (effects (font (size 1.27 1.27)) hide)
     )
@@
       (effects (font (size 1.27 1.27)) (justify left))
     )
-    (property "Footprint" "" (at 35.56 55.88 0)
+    (property "Footprint" "Resistor_SMD:R_0402_1005Metric" (at 35.56 55.88 0)
       (effects (font (size 1.27 1.27)) hide)
     )
@@
       (effects (font (size 1.27 1.27)))
     )
-    (property "Footprint" "" (at 218.44 119.38 0)
+    (property "Footprint" "Resistor_SMD:R_0402_1005Metric" (at 218.44 119.38 0)
       (effects (font (size 1.27 1.27)) hide)
     )
@@
       (effects (font (size 1.27 1.27)) (justify left))
     )
-    (property "Footprint" "" (at 223.52 83.82 0)
+    (property "Footprint" "Resistor_SMD:R_0402_1005Metric" (at 223.52 83.82 0)
       (effects (font (size 1.27 1.27)) hide)
     )
@@
       (effects (font (size 1.27 1.27)) (justify left))
     )
-    (property "Footprint" "" (at 223.52 114.3 0)
+    (property "Footprint" "Resistor_SMD:R_0402_1005Metric" (at 223.52 114.3 0)
       (effects (font (size 1.27 1.27)) hide)
     )
@@
       (effects (font (size 1.27 1.27)) (justify right))
     )
-    (property "Footprint" "" (at 259.08 114.3 0)
+    (property "Footprint" "Resistor_SMD:R_0402_1005Metric" (at 259.08 114.3 0)
       (effects (font (size 1.27 1.27)) hide)
     )
@@
       (effects (font (size 1.27 1.27)))
     )
-    (property "Footprint" "" (at 124.46 119.38 0)
+    (property "Footprint" "Resistor_SMD:R_0402_1005Metric" (at 124.46 119.38 0)
       (effects (font (size 1.27 1.27)) hide)
     )
@@
       (effects (font (size 1.27 1.27)))
     )
-    (property "Footprint" "" (at 124.46 60.96 0)
+    (property "Footprint" "Resistor_SMD:R_0402_1005Metric" (at 124.46 60.96 0)
       (effects (font (size 1.27 1.27)) hide)
     )
@@
       (effects (font (size 1.27 1.27)))
     )
-    (property "Footprint" "" (at 170.18 60.96 0)
+    (property "Footprint" "Resistor_SMD:R_0402_1005Metric" (at 170.18 60.96 0)
       (effects (font (size 1.27 1.27)) hide)
     )
@@
       (effects (font (size 1.27 1.27)))
     )
-    (property "Footprint" "" (at 218.44 88.9 0)
+    (property "Footprint" "Resistor_SMD:R_0402_1005Metric" (at 218.44 88.9 0)
       (effects (font (size 1.27 1.27)) hide)
     )
@@
       (effects (font (size 1.27 1.27)) (justify left))
     )
-    (property "Footprint" "" (at 129.54 83.82 0)
+    (property "Footprint" "Resistor_SMD:R_0402_1005Metric" (at 129.54 83.82 0)
       (effects (font (size 1.27 1.27)) hide)
     )
@@
       (effects (font (size 1.27 1.27)) (justify left))
     )
-    (property "Footprint" "" (at 35.56 25.4 0)
+    (property "Footprint" "Resistor_SMD:R_0402_1005Metric" (at 35.56 25.4 0)
       (effects (font (size 1.27 1.27)) hide)
     )
@@
       (effects (font (size 1.27 1.27)))
     )
-    (property "Footprint" "" (at 30.48 119.38 0)
+    (property "Footprint" "Resistor_SMD:R_0402_1005Metric" (at 30.48 119.38 0)
       (effects (font (size 1.27 1.27)) hide)
     )
@@
       (effects (font (size 1.27 1.27)))
     )
-    (property "Footprint" "" (at 124.46 88.9 0)
+    (property "Footprint" "Resistor_SMD:R_0402_1005Metric" (at 124.46 88.9 0)
       (effects (font (size 1.27 1.27)) hide)
     )

Commit message: feat: hardware: Assigns footprints for AD8066ARZ op amp and encoders
Parts:
- ENC1, ENC2, ENC3, ENC4, ENC5, ENC6: footprint PEC11R4220FS0024 -> Rotary_Encoder:PEC11R4220FS0024
Changed lines of the file:
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@@
       (effects (font (size 1.27 1.27)) (justify right))
     )
-    (property "Footprint" "PEC11R4220FS0024" (at 250.19 193.98 0)
+    (property "Footprint" "Rotary_Encoder:PEC11R4220FS0024" (at 250.19 193.98 0)
       (effects (font (size 1.27 1.27)) (justify left top) hide)
     )
@@
       (effects (font (size 1.27 1.27)) (justify right))
     )
-    (property "Footprint" "PEC11R4220FS0024" (at 62.23 135.56 0)
+    (property "Footprint" "Rotary_Encoder:PEC11R4220FS0024" (at 62.23 135.56 0)
       (effects (font (size 1.27 1.27)) (justify left top) hide)
     )
@@
       (effects (font (size 1.27 1.27)) (justify right))
     )
-    (property "Footprint" "PEC11R4220FS0024" (at 250.19 135.56 0)
+    (property "Footprint" "Rotary_Encoder:PEC11R4220FS0024" (at 250.19 135.56 0)
       (effects (font (size 1.27 1.27)) (justify left top) hide)
     )
@@
       (effects (font (size 1.27 1.27)) (justify right))
     )
-    (property "Footprint" "PEC11R4220FS0024" (at 156.21 193.98 0)
+    (property "Footprint" "Rotary_Encoder:PEC11R4220FS0024" (at 156.21 193.98 0)
       (effects (font (size 1.27 1.27)) (justify left top) hide)
     )
@@
       (effects (font (size 1.27 1.27)) (justify right))
     )
-    (property "Footprint" "PEC11R4220FS0024" (at 156.21 135.56 0)
+    (property "Footprint" "Rotary_Encoder:PEC11R4220FS0024" (at 156.21 135.56 0)
       (effects (font (size 1.27 1.27)) (justify left top) hide)
     )
@@
       (effects (font (size 1.27 1.27)) (justify right))
     )
-    (property "Footprint" "PEC11R4220FS0024" (at 62.23 193.98 0)
+    (property "Footprint" "Rotary_Encoder:PEC11R4220FS0024" (at 62.23 193.98 0)
       (effects (font (size 1.27 1.27)) (justify left top) hide)
     )

Commit message: feat: hardware: Assigns footprints for caps #3
Parts:
- C? (x6): footprint (none) -> Capacitor_SMD:C_0805_2012Metric
Changed lines of the file:
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@@
       (effects (font (size 1.27 1.27)) (justify right))
     )
-    (property "Footprint" "" (at 25.4 38.1 0)
+    (property "Footprint" "Capacitor_SMD:C_0805_2012Metric" (at 25.4 38.1 0)
       (effects (font (size 1.27 1.27)) hide)
     )
@@
       (effects (font (size 1.27 1.27)) (justify right))
     )
-    (property "Footprint" "" (at 213.36 35.56 0)
+    (property "Footprint" "Capacitor_SMD:C_0805_2012Metric" (at 213.36 35.56 0)
       (effects (font (size 1.27 1.27)) hide)
     )
@@
       (effects (font (size 1.27 1.27)) (justify right))
     )
-    (property "Footprint" "" (at 119.38 93.98 0)
+    (property "Footprint" "Capacitor_SMD:C_0805_2012Metric" (at 119.38 93.98 0)
       (effects (font (size 1.27 1.27)) hide)
     )
@@
       (effects (font (size 1.27 1.27)) (justify right))
     )
-    (property "Footprint" "" (at 213.36 93.98 0)
+    (property "Footprint" "Capacitor_SMD:C_0805_2012Metric" (at 213.36 93.98 0)
       (effects (font (size 1.27 1.27)) hide)
     )
@@
       (effects (font (size 1.27 1.27)) (justify right))
     )
-    (property "Footprint" "" (at 25.4 93.98 0)
+    (property "Footprint" "Capacitor_SMD:C_0805_2012Metric" (at 25.4 93.98 0)
       (effects (font (size 1.27 1.27)) hide)
     )
@@
       (effects (font (size 1.27 1.27)) (justify right))
     )
-    (property "Footprint" "" (at 119.38 35.56 0)
-      (effects (font (size 1.27 1.27)) hide)
-    )
+    (property "Footprint" "Capacitor_SMD:C_0805_2012Metric" (at 119.38 35.56 0)
+      (effects (font (size 1.27 1.27)) hide)
+    )
