File: hardware/kicad/tinyscope/hmi.kicad_sch (KiCad schematic)
At the start: 61 parts, among them J8 Waveshare 16498

Commit message: feat: hardware: Assigns footprints for connectors #1
Parts:
- J8: footprint (none) -> Connector_PinSocket_2.54mm:PinSocket_2x17_P2.54mm_Vertical_SMD
Changed lines of the file:
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@@
       (effects (font (size 1.27 1.27)))
     )
-    (property "Footprint" "" (at 63.5 167.64 0)
+    (property "Footprint" "Connector_PinSocket_2.54mm:PinSocket_2x17_P2.54mm_Vertical_SMD" (at 63.5 167.64 0)
       (effects (font (size 1.27 1.27)) hide)
     )
