File: hardware/kicad/tinyscope/regulation_and_rails.kicad_sch (KiCad schematic)
At the start: 28 parts

Commit message: feat: hardware: Assigns footprints for TPS63802DLAR voltage regulator and MAX17048 fuel gauge
Parts:
- U? (x2): footprint TPS63802DLAR -> Package_SON:TPS63802DLAR
Changed lines of the file:
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@@
       (effects (font (size 1.27 1.27)))
     )
-    (property "Footprint" "TPS63802DLAR" (at 88.9 206.68 0)
+    (property "Footprint" "Package_SON:TPS63802DLAR" (at 88.9 206.68 0)
       (effects (font (size 1.27 1.27)) (justify left top) hide)
     )
@@
       (effects (font (size 1.27 1.27)))
     )
-    (property "Footprint" "TPS63802DLAR" (at 88.9 148.26 0)
+    (property "Footprint" "Package_SON:TPS63802DLAR" (at 88.9 148.26 0)
       (effects (font (size 1.27 1.27)) (justify left top) hide)
     )

Commit message: feat: hardware: Assigns footprints for caps #3
Parts:
- C? (x9): footprint (none) -> Capacitor_SMD:C_1210_3225Metric
- C? (x2): footprint (none) -> Capacitor_SMD:CP_Elec_6.3x5.7
- C?: footprint (none) -> Capacitor_SMD:C_0805_2012Metric
Changed lines of the file:
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@@
       (effects (font (size 1.27 1.27)) (justify right))
     )
-    (property "Footprint" "" (at 153.67 62.23 0)
+    (property "Footprint" "Capacitor_SMD:C_1210_3225Metric" (at 153.67 62.23 0)
       (effects (font (size 1.27 1.27)) hide)
     )
@@
       (effects (font (size 1.27 1.27)) (justify left))
     )
-    (property "Footprint" "" (at 110.49 58.42 0)
+    (property "Footprint" "Capacitor_SMD:CP_Elec_6.3x5.7" (at 110.49 58.42 0)
       (effects (font (size 1.27 1.27)) hide)
     )
@@
       (effects (font (size 1.27 1.27)) (justify left))
     )
-    (property "Footprint" "" (at 203.2 60.96 0)
+    (property "Footprint" "Capacitor_SMD:C_1210_3225Metric" (at 203.2 60.96 0)
       (effects (font (size 1.27 1.27)) hide)
     )
@@
       (effects (font (size 1.27 1.27)) (justify right))
     )
-    (property "Footprint" "" (at 143.51 55.88 0)
+    (property "Footprint" "Capacitor_SMD:C_1210_3225Metric" (at 143.51 55.88 0)
       (effects (font (size 1.27 1.27)) hide)
     )
@@
       (effects (font (size 1.27 1.27)) (justify left))
     )
-    (property "Footprint" "" (at 161.29 119.38 0)
+    (property "Footprint" "Capacitor_SMD:C_0805_2012Metric" (at 161.29 119.38 0)
       (effects (font (size 1.27 1.27)) hide)
     )
@@
       (effects (font (size 1.27 1.27)) (justify right))
     )
-    (property "Footprint" "" (at 41.91 60.96 0)
+    (property "Footprint" "Capacitor_SMD:C_1210_3225Metric" (at 41.91 60.96 0)
       (effects (font (size 1.27 1.27)) hide)
     )
@@
       (effects (font (size 1.27 1.27)) (justify right))
     )
-    (property "Footprint" "" (at 41.91 119.38 0)
+    (property "Footprint" "Capacitor_SMD:C_1210_3225Metric" (at 41.91 119.38 0)
       (effects (font (size 1.27 1.27)) hide)
     )
@@
       (effects (font (size 1.27 1.27)) (justify left))
     )
-    (property "Footprint" "" (at 186.69 119.38 0)
+    (property "Footprint" "Capacitor_SMD:C_1210_3225Metric" (at 186.69 119.38 0)
       (effects (font (size 1.27 1.27)) hide)
     )
@@
       (effects (font (size 1.27 1.27)) (justify right))
     )
-    (property "Footprint" "" (at 236.22 63.5 0)
-      (effects (font (size 1.27 1.27)) hide)
-    )
-    (property "Datasheet" "~" (at 236.22 63.5 0)
+    (property "Footprint" "Capacitor_SMD:C_1210_3225Metric" (at 236.22 63.5 0)
+      (effects (font (size 1.27 1.27)) hide)
+    )
+    (property "Datasheet" "https://www.mouser.pl/en/ProductDetail/Wurth-Elektronik/865080643008?qs=sGAEpiMZZMsh%252B1woXyUXj4jKQI6sNRw6T99VCXuPOwI%3D" (at 236.22 63.5 0)
       (effects (font (size 1.27 1.27)) hide)
     )
@@
       (effects (font (size 1.27 1.27)) (justify left))
     )
-    (property "Footprint" "" (at 119.38 116.84 0)
+    (property "Footprint" "Capacitor_SMD:CP_Elec_6.3x5.7" (at 119.38 116.84 0)
       (effects (font (size 1.27 1.27)) hide)
     )
@@
       (effects (font (size 1.27 1.27)) (justify left))
     )
-    (property "Footprint" "" (at 276.86 63.5 0)
-      (effects (font (size 1.27 1.27)) hide)
-    )
-    (property "Datasheet" "~" (at 276.86 63.5 0)
+    (property "Footprint" "Capacitor_SMD:C_1210_3225Metric" (at 276.86 63.5 0)
+      (effects (font (size 1.27 1.27)) hide)
+    )
+    (property "Datasheet" "https://www.mouser.pl/en/ProductDetail/Wurth-Elektronik/865080643008?qs=sGAEpiMZZMsh%252B1woXyUXj4jKQI6sNRw6T99VCXuPOwI%3D" (at 276.86 63.5 0)
       (effects (font (size 1.27 1.27)) hide)
     )
@@
       (effects (font (size 1.27 1.27)) (justify left))
     )
-    (property "Footprint" "" (at 181.61 68.58 0)
-      (effects (font (size 1.27 1.27)) hide)
-    )
+    (property "Footprint" "Capacitor_SMD:C_1210_3225Metric" (at 181.61 68.58 0)
+      (effects (font (size 1.27 1.27)) hide)
+    )

Commit message: feat: hardware: Assigns footprints for caps #4
Parts:
- C? (x4): footprint Capacitor_SMD:C_1210_3225Metric -> Capacitor_SMD:C_0805_2012Metric
- C? (x2): footprint Capacitor_SMD:CP_Elec_6.3x5.7 -> Capacitor_SMD:C_0603_1608Metric
- C? (x2): footprint Capacitor_SMD:C_1210_3225Metric -> Capacitor_SMD:C_0603_1608Metric
- C?: footprint (none) -> Capacitor_SMD:C_0805_2012Metric
- L? (x2): footprint (none) -> Inductor_SMD:L_1008_2520Metric
Changed lines of the file:
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@@
       (effects (font (size 1.27 1.27)) (justify right))
     )
-    (property "Footprint" "Capacitor_SMD:C_1210_3225Metric" (at 153.67 62.23 0)
-      (effects (font (size 1.27 1.27)) hide)
-    )
-    (property "Datasheet" "~" (at 153.67 62.23 0)
+    (property "Footprint" "Capacitor_SMD:C_0805_2012Metric" (at 153.67 62.23 0)
+      (effects (font (size 1.27 1.27)) hide)
+    )
+    (property "Datasheet" "https://www.mouser.pl/en/ProductDetail/KYOCERA-AVX/KGM21AR71C105JU?qs=sGAEpiMZZMuMW9TJLBQkXqLYvz3DzaXfu86Idg8N2os%3D" (at 153.67 62.23 0)
       (effects (font (size 1.27 1.27)) hide)
     )
@@
       (effects (font (size 1.27 1.27)) (justify left))
     )
-    (property "Footprint" "Capacitor_SMD:CP_Elec_6.3x5.7" (at 110.49 58.42 0)
+    (property "Footprint" "Capacitor_SMD:C_0603_1608Metric" (at 110.49 58.42 0)
       (effects (font (size 1.27 1.27)) hide)
     )
@@
       (effects (font (size 1.27 1.27)) (justify left))
     )
-    (property "Footprint" "" (at 100.33 116.84 0)
-      (effects (font (size 1.27 1.27)) hide)
-    )
-    (property "Datasheet" "~" (at 100.33 116.84 0)
+    (property "Footprint" "Inductor_SMD:L_1008_2520Metric" (at 100.33 116.84 0)
+      (effects (font (size 1.27 1.27)) hide)
+    )
+    (property "Datasheet" "https://www.mouser.pl/en/ProductDetail/Bourns/SRP2512PA-R47M?qs=sGAEpiMZZMv126LJFLh8y4TWbsvnEkXNffWcaB1Qgxk%3D" (at 100.33 116.84 0)
       (effects (font (size 1.27 1.27)) hide)
     )
@@
       (effects (font (size 1.27 1.27)) (justify left))
     )
-    (property "Footprint" "Capacitor_SMD:C_1210_3225Metric" (at 203.2 60.96 0)
-      (effects (font (size 1.27 1.27)) hide)
-    )
-    (property "Datasheet" "~" (at 203.2 60.96 0)
+    (property "Footprint" "Capacitor_SMD:C_0805_2012Metric" (at 203.2 60.96 0)
+      (effects (font (size 1.27 1.27)) hide)
+    )
+    (property "Datasheet" "https://www.mouser.pl/en/ProductDetail/Murata-Electronics/GCJ21BR71E225KA01K?qs=QzBtWTOodeVaagW24xxz2w%3D%3D" (at 203.2 60.96 0)
       (effects (font (size 1.27 1.27)) hide)
     )
@@
       (effects (font (size 1.27 1.27)) (justify right))
     )
-    (property "Footprint" "Capacitor_SMD:C_1210_3225Metric" (at 143.51 55.88 0)
-      (effects (font (size 1.27 1.27)) hide)
-    )
-    (property "Datasheet" "~" (at 143.51 55.88 0)
+    (property "Footprint" "Capacitor_SMD:C_0805_2012Metric" (at 143.51 55.88 0)
+      (effects (font (size 1.27 1.27)) hide)
+    )
+    (property "Datasheet" "https://www.mouser.pl/en/ProductDetail/Murata-Electronics/GXT21BR71A475KE13L?qs=sGAEpiMZZMuMW9TJLBQkXh6n3NgygzPJ8oec6baIqTc%3D" (at 143.51 55.88 0)
       (effects (font (size 1.27 1.27)) hide)
     )
@@
       (effects (font (size 1.27 1.27)) (justify left))
     )
-    (property "Footprint" "" (at 100.33 58.42 0)
-      (effects (font (size 1.27 1.27)) hide)
-    )
-    (property "Datasheet" "~" (at 100.33 58.42 0)
+    (property "Footprint" "Inductor_SMD:L_1008_2520Metric" (at 100.33 58.42 0)
+      (effects (font (size 1.27 1.27)) hide)
+    )
+    (property "Datasheet" "https://www.mouser.pl/en/ProductDetail/Bourns/SRP2512PA-R47M?qs=sGAEpiMZZMv126LJFLh8y4TWbsvnEkXNffWcaB1Qgxk%3D" (at 100.33 58.42 0)
       (effects (font (size 1.27 1.27)) hide)
     )
@@
       (effects (font (size 1.27 1.27)) (justify right))
     )
-    (property "Footprint" "Capacitor_SMD:C_1210_3225Metric" (at 41.91 60.96 0)
+    (property "Footprint" "Capacitor_SMD:C_0603_1608Metric" (at 41.91 60.96 0)
       (effects (font (size 1.27 1.27)) hide)
     )
@@
       (effects (font (size 1.27 1.27)) (justify right))
     )
-    (property "Footprint" "Capacitor_SMD:C_1210_3225Metric" (at 41.91 119.38 0)
+    (property "Footprint" "Capacitor_SMD:C_0603_1608Metric" (at 41.91 119.38 0)
       (effects (font (size 1.27 1.27)) hide)
     )
@@
       (effects (font (size 1.27 1.27)) hide)
     )
-    (property "Datasheet" "https://www.mouser.pl/en/ProductDetail/Wurth-Elektronik/865080643008?qs=sGAEpiMZZMsh%252B1woXyUXj4jKQI6sNRw6T99VCXuPOwI%3D" (at 236.22 63.5 0)
+    (property "Datasheet" "" (at 236.22 63.5 0)
       (effects (font (size 1.27 1.27)) hide)
     )
@@
       (effects (font (size 1.27 1.27)) (justify left))
     )
-    (property "Footprint" "Capacitor_SMD:CP_Elec_6.3x5.7" (at 119.38 116.84 0)
+    (property "Footprint" "Capacitor_SMD:C_0603_1608Metric" (at 119.38 116.84 0)
       (effects (font (size 1.27 1.27)) hide)
     )
@@
       (effects (font (size 1.27 1.27)) (justify left))
     )
-    (property "Footprint" "Capacitor_SMD:C_1210_3225Metric" (at 181.61 68.58 0)
-      (effects (font (size 1.27 1.27)) hide)
-    )
-    (property "Datasheet" "~" (at 181.61 68.58 0)
+    (property "Footprint" "Capacitor_SMD:C_0805_2012Metric" (at 181.61 68.58 0)
+      (effects (font (size 1.27 1.27)) hide)
+    )
+    (property "Datasheet" "https://www.mouser.pl/en/ProductDetail/Murata-Electronics/GXT21BR71A475KE13L?qs=sGAEpiMZZMuMW9TJLBQkXh6n3NgygzPJ8oec6baIqTc%3D" (at 181.61 68.58 0)
       (effects (font (size 1.27 1.27)) hide)
     )
@@
       (effects (font (size 1.27 1.27)) (justify left))
     )
-    (property "Footprint" "" (at 266.7 68.58 0)
-      (effects (font (size 1.27 1.27)) hide)
-    )
+    (property "Footprint" "Capacitor_SMD:C_0805_2012Metric" (at 266.7 68.58 0)
+      (effects (font (size 1.27 1.27)) hide)
+    )

Commit message: feat: hardware: Finishes footprints selection for ADP7142 LDO
Parts:
- C? (x2): footprint Capacitor_SMD:C_1210_3225Metric -> Capacitor_SMD:C_0805_2012Metric
Changed lines of the file:
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@@
       (effects (font (size 1.27 1.27)) (justify right))
     )
-    (property "Footprint" "Capacitor_SMD:C_1210_3225Metric" (at 236.22 63.5 0)
+    (property "Footprint" "Capacitor_SMD:C_0805_2012Metric" (at 236.22 63.5 0)
       (effects (font (size 1.27 1.27)) hide)
     )
-    (property "Datasheet" "" (at 236.22 63.5 0)
+    (property "Datasheet" "https://www.mouser.pl/en/ProductDetail/Murata-Electronics/GCJ21BR71E225KA01K?qs=QzBtWTOodeVaagW24xxz2w%3D%3D" (at 236.22 63.5 0)
       (effects (font (size 1.27 1.27)) hide)
     )
@@
       (effects (font (size 1.27 1.27)) (justify left))
     )
-    (property "Footprint" "Capacitor_SMD:C_1210_3225Metric" (at 276.86 63.5 0)
+    (property "Footprint" "Capacitor_SMD:C_0805_2012Metric" (at 276.86 63.5 0)
       (effects (font (size 1.27 1.27)) hide)
     )
-    (property "Datasheet" "https://www.mouser.pl/en/ProductDetail/Wurth-Elektronik/865080643008?qs=sGAEpiMZZMsh%252B1woXyUXj4jKQI6sNRw6T99VCXuPOwI%3D" (at 276.86 63.5 0)
+    (property "Datasheet" "https://www.mouser.pl/en/ProductDetail/Murata-Electronics/GCJ21BR71E225KA01K?qs=QzBtWTOodeVaagW24xxz2w%3D%3D" (at 276.86 63.5 0)
       (effects (font (size 1.27 1.27)) hide)
     )

Commit message: feat: hardware: Finishes footprints selection for REF3030 voltage reference
Parts:
- C?: footprint Capacitor_SMD:C_0805_2012Metric -> Capacitor_SMD:C_0603_1608Metric
- C?: footprint Capacitor_SMD:C_1210_3225Metric -> Capacitor_SMD:C_0805_2012Metric
Changed lines of the file:
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@@
       (effects (font (size 1.27 1.27)) (justify left))
     )
-    (property "Footprint" "Capacitor_SMD:C_0805_2012Metric" (at 161.29 119.38 0)
-      (effects (font (size 1.27 1.27)) hide)
-    )
-    (property "Datasheet" "~" (at 161.29 119.38 0)
+    (property "Footprint" "Capacitor_SMD:C_0603_1608Metric" (at 161.29 119.38 0)
+      (effects (font (size 1.27 1.27)) hide)
+    )
+    (property "Datasheet" "https://www.mouser.pl/en/ProductDetail/Murata-Electronics/GCM188R71H104KA57D?qs=aEuGZpxfbxWuy5eQGqiN%252BA%3D%3D" (at 161.29 119.38 0)
       (effects (font (size 1.27 1.27)) hide)
     )
@@
       (effects (font (size 1.27 1.27)) (justify left))
     )
-    (property "Footprint" "Capacitor_SMD:C_1210_3225Metric" (at 186.69 119.38 0)
-      (effects (font (size 1.27 1.27)) hide)
-    )
-    (property "Datasheet" "~" (at 186.69 119.38 0)
-      (effects (font (size 1.27 1.27)) hide)
-    )
+    (property "Footprint" "Capacitor_SMD:C_0805_2012Metric" (at 186.69 119.38 0)
+      (effects (font (size 1.27 1.27)) hide)
+    )
+    (property "Datasheet" "https://www.mouser.pl/en/ProductDetail/Murata-Electronics/GCG21BR71E105JA12K?qs=QzBtWTOodeWowTZRO4rL3w%3D%3D" (at 186.69 119.38 0)
+      (effects (font (size 1.27 1.27)) hide)
+    )
